File: Kicad/Computer/SNES Device/SNES Device Selector.kicad_sch (KiCad schematic)
At the start: 16 parts, among them IC25 74LVC1G08GV,125, IC26 74LVC2G32DP,125, IC27 74LVC1G02GV,125, IC28 74LVC273PW,118, IC29 74ALVC32PW,118, IC30 74ALVC32PW,118, IC31 74LVC541APW,118, IC32 74LVC541APW,118

Commit message: Split SNES device into multiple boards.
Connections:
- no-connect marks 0 -> 2
Changed lines of the file:
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@@
   (junction (at 193.04 107.95) (diameter 0) (color 0 0 0 0)
   )
+  (no_connect (at 39.37 45.72))
+  (no_connect (at 39.37 40.64))
   (bus_entry (at 231.14 118.11) (size 2.54 2.54)
     (stroke (width 0) (type default) (color 0 0 0 0))
@@
     (effects (font (size 1.27 1.27)) (justify left bottom))
   )
-  (label "~{Select3}" (at 39.37 45.72 0)
-    (effects (font (size 1.27 1.27)) (justify left bottom))
-  )
   (label "GND" (at 265.43 85.09 0)
     (effects (font (size 1.27 1.27)) (justify left bottom))
@@
     (effects (font (size 1.27 1.27)) (justify left bottom))
   )
-  (label "~{Select1}" (at 39.37 40.64 0)
-    (effects (font (size 1.27 1.27)) (justify left bottom))
-  )
