File: Kicad/Computer/Clock/Clock.kicad_sch (KiCad schematic)
At the start: 55 parts, among them IC1 74VHC393FT, IC10 SN74ABT245BDBR, IC2 MC74VHC139DR2G, IC3 74VHC595FT, IC4 74VHC74M, IC5 DS1813R, IC6 MC74VHC04DR2G, IC7 74AHC125S14, IC8 74AHC125S14, IC9 SN74ABT245BDBR, J1 Conn_01x06_Male, J2 Conn_01x12_Male, J3 Conn_01x06_Male, J4 Conn_01x12_Male

Commit message: Redoing Clock PCB from scratch.
Parts:
- removed C1: LMK325ABJ107MM-P, CAPC3225X270N, symbol Taiyo_Yuden:LMK325ABJ107MM-P
- removed C11, C9: CL21A106KPFNNNF, CAPC2012X135N, symbol Samsung:CL21A106KPFNNNF
- removed IC7, IC8: 74AHC125S14, SOIC127P600X173-14N, symbol Diodes_Inc:74AHC125S14-13
- removed J1, J3: Conn_01x06_Male, Connector_PinHeader_2.54mm:PinHeader_1x06_P2.54mm_Vertical, symbol Connector:Conn_01x06_Male
- added C1, C2, C3, C4, C5: C_Small, Capacitor_SMD:C_0805_2012Metric, symbol Device:C_Small
- added IC10, IC9: 74AHC125S14, SOIC127P600X173-14N, symbol Diodes_Inc:74AHC125S14
- added J1, J10, J12, J3, J4, J6, J7, J9: Conn_01x02_Male, Connector_PinHeader_2.54mm:PinHeader_1x02_P2.54mm_Vertical, symbol Connector:Conn_01x02_Male
- added J2, J5: Conn_01x04_Male, Connector_PinHeader_2.54mm:PinHeader_1x04_P2.54mm_Vertical, symbol Connector:Conn_01x04_Male
- added NT2: NetTie_2, NetTie:NetTie-2_SMD_Pad0.5mm, symbol Device:NetTie_2
- added PS1: AP2210K-5.0TRG1, SOT95P282X130-5N, symbol Diodes_Inc:AP2210K-5.0TRG1
- added R5, R6, R7, R8, R9: R_Small, Resistor_SMD:R_0805_2012Metric, symbol Device:R_Small
- IC1: renamed from IC5; value DS1813R -> DS1813R-10+T&R
- R1: renamed from R4; Resistance 47Ω -> (none)
- R11: renamed from R8; Resistance 680Ω -> (none)
- R12: renamed from R2; Resistance 680Ω -> (none)
- R13: renamed from R3; Resistance 680Ω -> (none)
- R2: renamed from R7; Resistance 47Ω -> (none)
- R3: renamed from R5; Resistance 47Ω -> (none)
- R4: renamed from R6; Resistance 47Ω -> (none)
- renumbered C6 to C10, C7 to C11, C8 to C12, C10 to C13, C12 to C14, C2 to C6, C3 to C7, C4 to C8, C5 to C9, IC3 to IC2, IC4 to IC3, IC6 to IC4, IC9 to IC5, IC1 to IC6, IC10 to IC7, IC2 to IC8, J4 to J11, J2 to J8, LED12 to LED10, LED13 to LED11, LED14 to LED12, LED15 to LED13, LED9 to LED14, LED10 to LED15, LED11 to LED9, R1 to R10, RN2 to RN1, RN3 to RN2, RN4 to RN3, RN1 to RN4
Connections:
- net Clock: now also IC6.13 (2~{CK})
- net Count 1 A: now also R7.2; no longer IC6.3 (1QA)
- net Count 1 B: now also R6.2; no longer IC6.4 (1QB)
- net Count 1 D: now also R5.2; no longer IC6.6 (1QD)
- net Count 2 A: now also R9.2; no longer IC6.11 (2QA)
- net Count 2 B: now also R8.2; no longer IC6.10 (2QB)
- net GND: now also C1.1, C2.1, C3.1, C4.1, C5.1, IC10.1 (1~{OE}), IC10.10 (3~{OE}), IC10.13 (4~{OE}), IC10.4 (2~{OE}), IC10.7 (GND), IC9.1 (1~{OE}), IC9.10 (3~{OE}), IC9.13 (4~{OE}), IC9.4 (2~{OE}), IC9.7 (GND), J1.1 (Pin_1), J10.1 (Pin_1), J12.1 (Pin_1), J3.1 (Pin_1), J4.1 (Pin_1), J6.1 (Pin_1), J7.1 (Pin_1), J9.1 (Pin_1), PS1.2 (GND)
- net Reset Switch: now also J2.4 (Pin_4), J5.4 (Pin_4)
- net Source Clock: now also J2.2 (Pin_2), J5.2 (Pin_2)
- net ~{Clock}: now also IC3.2 (D1), IC6.1 (1~{CK})
- net ~{Reset} GND: now also J2.3 (Pin_3), J5.3 (Pin_3)
- net at IC3.6 (~{Q1}), R4.1: no longer IC3.2 (D1), IC6.1 (1~{CK})
- net at RN4.7: now also IC9.3 (1Y)
- net at IC8.7 (~{Y3A}): now also IC9.2 (1A)
- net at IC8.4 (~{Y0A}): now also IC9.12 (4A)
- net at RN4.1: now also IC9.11 (4Y)
- net at IC8.5 (~{Y1A}): now also IC9.9 (3A)
- net at RN4.3: now also IC9.8 (3Y)
- net at RN4.5: now also IC9.6 (2Y)
- net at IC8.6 (~{Y2A}): now also IC9.5 (2A)
- net at RN4.8: now also IC10.11 (4Y)
- net at IC8.9 (~{Y3B}): now also IC10.2 (1A)
- net at IC8.12 (~{Y0B}): now also IC10.12 (4A)
- net at RN4.2: now also IC10.3 (1Y)
- net at IC8.11 (~{Y1B}): now also IC10.9 (3A)
- net at RN4.4: now also IC10.6 (2Y)
- net at RN4.6: now also IC10.8 (3Y)
- net at IC8.10 (~{Y2B}): now also IC10.5 (2A)
- net at IC3.5 (Q1), R3.1: no longer IC6.13 (2~{CK})
- net Reset LED: now reaches LED14.2
- net Reset LED: now also IC4.12 (6Y); no longer IC4.6 (~{Y3})
- net Reset Switch LED: now reaches LED15.2
- net Reset Switch LED: now also IC4.6 (3Y); no longer IC4.12 (~{Y6})
- net 5V renamed VCC
- net VCC: now also C3.2, C4.2, C5.2, IC10.14 (VCC), IC9.14 (VCC), NT2.1, PS1.5 (VOUT); no longer LED13.2
- new net: J2.1 (Pin_1), J5.1 (Pin_1)
- new net: IC6.6 (1QD), R5.1
- new net: IC6.11 (2QA), R9.1
- new net: IC6.4 (1QB), R6.1
- new net: C2.2, PS1.4 (BYP)
- new net: IC6.10 (2QB), R8.1
- new net: IC6.3 (1QA), R7.1
- new net Power LED: LED13.2, NT2.2
- new net Source 5V: C1.2, J1.2 (Pin_2), J10.2 (Pin_2), J12.2 (Pin_2), J3.2 (Pin_2), J4.2 (Pin_2), J6.2 (Pin_2), J7.2 (Pin_2), J9.2 (Pin_2), PS1.1 (VIN), PS1.3 (EN)
- no-connect marks 14 -> 15
Other:
- moved on the sheet: C10, C11, C12, C13, C14, C6, C7, C8, C9, IC5, IC6, IC7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

Commit message: Laying out ancillary ICs.
Parts:
- renumbered LED10 to LD10, LED11 to LD11, LED12 to LD12, LED13 to LD13, LED14 to LD14, LED15 to LD15
Connections:
- net at LED8.1: now also RN2.1 (R1_1); no longer RN2.4 (R4_1)
- net at LED5.1: now also RN2.4 (R4_1); no longer RN2.1 (R1_1)
- net at LED3.1: now also RN1.2 (R2_1); no longer RN1.3 (R3_1)
- net at LED4.1: now also RN1.1 (R1_1); no longer RN1.4 (R4_1)
- net at LED2.1: now also RN1.3 (R3_1); no longer RN1.2 (R2_1)
- net at RN2.2 (R2_1): now also LED7.1; no longer LED6.1
- net at RN2.3 (R3_1): now also LED6.1; no longer LED7.1
- net at LED1.1: now also RN1.4 (R4_1); no longer RN1.1 (R1_1)

Commit message: Laid out Clock but not ancillary PCB.
Parts:
- removed LD10, LD11, LD12, LED9: 150224VS73100A, 150224VS73100A, symbol Wurth_Elektronik:150224VS73100A
- removed R11, R12, R13, R2, R3, R4, R6, R7, R8, R9: R_Small, Resistor_SMD:R_0805_2012Metric, symbol Device:R_Small
- removed RN1, RN2, RN3: CAY16-472J4LF, CAY16472J4LF, symbol Bourns:CAY16-472J4LF
- removed RN4: 4816P-1-470LF, SOIC127P762X240-16N, symbol Bourns:4816P-1-470LF
- added LD10, LD11, LD12, LED9: 150224BS73100A, 150224BS73100A, symbol Wurth_Elektronik:150224BS73100A
- added RN1, RN2: CAY16-681J4LF, SamacSys_Parts:CAY16-J4, symbol Bourns:CAY16-681J4LF
- added RN3: CAY16-103J4LF, SamacSys_Parts:CAY16-J4, symbol Bourns:CAY16-103J4LF
- added RN4, RN5, RN6, RN8: CAY16-470J4LF, CAY16470J4LF, symbol Bourns:CAY16-470J4LF
- added RN7: CAY16-102J4LF, SamacSys_Parts:CAY16-J4, symbol Bourns:CAY16-102J4LF
- C1, C10, C11, C12, C13, C14, C2, C3, C4, C5, C6, C7, C8, C9: footprint Capacitor_SMD:C_0805_2012Metric -> (none)
- IC1: Silkscreen (none) -> DS1813
- J1, J10, J12, J3, J4, J6, J7, J9: footprint Connector_PinHeader_2.54mm:PinHeader_1x02_P2.54mm_Vertical -> (none)
- J11, J8: footprint Connector_PinHeader_2.54mm:PinHeader_1x12_P2.54mm_Vertical -> (none)
- J2, J5: footprint Connector_PinHeader_2.54mm:PinHeader_1x04_P2.54mm_Vertical -> (none)
- LD13, LD14, LD15: footprint LEDM2314X131N -> SamacSys_Parts:150224SS73100A; Silkscreen (none) -> red
- LED1, LED2, LED3, LED4, LED5, LED6, LED7, LED8: Silkscreen (none) -> grn
- NT1, NT2: footprint NetTie:NetTie-2_SMD_Pad0.5mm -> (none)
- PS1: Silkscreen (none) -> AP2210K
- R1, R10, R5: footprint Resistor_SMD:R_0805_2012Metric -> (none)
Connections:
- net Clock: now also IC7.3 (A2), RN5.8 (R1); no longer IC7.17 (B2)
- net Count 1 A: now also RN6.7 (R2)
- net Count 1 B: now also RN6.8 (R1)
- net Count 2 A: now also RN6.5 (R4)
- net Count 2 B: now also RN6.6 (R3)
- net GND: now also C5.2, IC7.6 (A5), IC7.7 (A6), IC7.8 (A7), IC7.9 (A8), RN1.1 (R1), RN1.2 (R2), RN1.3 (R3), RN1.4 (R4), RN2.1 (R1), RN2.2 (R2), RN2.3 (R3), RN2.4 (R4), RN3.1 (R1), RN3.2 (R2), RN3.3 (R3), RN3.4 (R4), RN7.1 (R1), RN7.3 (R3), RN7.4 (R4); no longer C5.1, IC5.1 (DIR), IC7.1 (DIR), IC7.11 (B8), IC7.12 (B7), IC7.13 (B6), IC7.14 (B5)
- net Reset Switch: no longer IC1.1 (~{RST}), IC2.10 (~{SCLR}), IC2.14 (SI), IC4.5 (3A)
- net Slow Selector: now also IC7.5 (A4), RN5.6 (R3); no longer IC7.15 (B4)
- net Source 5V: no longer J1.2 (Pin_2), J10.2 (Pin_2), J12.2 (Pin_2), J4.2 (Pin_2), J7.2 (Pin_2), J9.2 (Pin_2)
- net Source Clock: now also IC7.2 (A1); no longer IC7.18 (B1)
- net VCC: now also C5.1, IC5.1 (DIR), IC7.1 (DIR); no longer C5.2
- net ~{Clock}: now also IC7.4 (A3), RN5.7 (R2); no longer IC7.16 (B3)
- net ~{Select 0}: now also IC5.2 (A1), RN4.5 (R4); no longer IC5.18 (B1)
- net ~{Select 1}: now also IC5.3 (A2), RN8.5 (R4); no longer IC5.17 (B2)
- net ~{Select 2}: now also IC5.4 (A3), RN4.6 (R3); no longer IC5.16 (B3)
- net ~{Select 3}: now also IC5.5 (A4), RN8.6 (R3); no longer IC5.15 (B4)
- net ~{Select 4}: now also IC5.6 (A5), RN4.7 (R2); no longer IC5.14 (B5)
- net ~{Select 5}: now also IC5.7 (A6), RN8.7 (R2); no longer IC5.13 (B6)
- net ~{Select 6}: now also IC5.8 (A7), RN4.8 (R1); no longer IC5.12 (B7)
- net ~{Select 7}: now also IC5.9 (A8), RN8.8 (R1); no longer IC5.11 (B8)
- net at LED1.2: now also IC5.18 (B1); no longer IC5.2 (A1)
- net at LED2.2: now also IC5.17 (B2); no longer IC5.3 (A2)
- net at LED3.2: now also IC5.16 (B3); no longer IC5.4 (A3)
- net at LED4.2: now also IC5.15 (B4); no longer IC5.5 (A4)
- net at LED5.2: now also IC5.14 (B5); no longer IC5.6 (A5)
- net at LED6.2: now also IC5.13 (B6); no longer IC5.7 (A6)
- net at LED7.2: now also IC5.12 (B7); no longer IC5.8 (A7)
- net at LED8.2: now also IC5.11 (B8); no longer IC5.9 (A8)
- net at LED8.1: now also RN2.5 (R4)
- net Count 1QD: now reaches IC6.6 (1QD), R5.1
- net Shift QA: now reaches IC2.15 (QA), R1.1
- net Shift QE: now reaches IC2.4 (QE), IC3.1 (~{CLR1}), IC3.13 (~{CLR2})
- net Shift QG: now reaches IC2.6 (QG), IC4.1 (1A)
- net Shift QH: now reaches IC2.7 (QH), IC4.3 (2A)
- net Flop ~{Q1}: now reaches IC3.6 (~{Q1})
- net Flop ~{Q1}: now also RN5.2 (R2)
- net Drive2 4Y: now reaches IC10.11 (4Y)
- net Drive2 4Y: now also RN8.4 (R4)
- net Line ~{Y0B}: now reaches IC10.12 (4A), IC8.12 (~{Y0B})
- net Line ~{Y3B}: now reaches IC10.2 (1A), IC8.9 (~{Y3B})
- net Drive2 1Y: now reaches IC10.3 (1Y)
- net Drive2 1Y: now also RN8.1 (R1)
- net Line ~{Y2B}: now reaches IC10.5 (2A), IC8.10 (~{Y2B})
- net Drive2 2Y: now reaches IC10.6 (2Y)
- net Drive2 2Y: now also RN8.2 (R2)
- net Drive2 3Y: now reaches IC10.8 (3Y)
- net Drive2 3Y: now also RN8.3 (R3)
- net Line ~{Y1B}: now reaches IC10.9 (3A), IC8.11 (~{Y1B})
- net Count 2QA: now reaches IC6.11 (2QA)
- net Count 2QA: now also RN6.4 (R4)
- net Flop Q2: now reaches IC3.9 (Q2)
- net Flop Q2: now also RN5.3 (R3)
- net at LD13.1: now also RN7.8 (R1)
- net at LED5.1: now also RN2.8 (R1)
- net Count 1QB: now reaches IC6.4 (1QB)
- net Count 1QB: now also RN6.1 (R1)
- net Flop D2: now reaches IC3.12 (D2)
- net Flop D2: now also RN5.5 (R4); no longer IC3.8 (~{Q2})
- net Flop Q1: now reaches IC3.5 (Q1)
- net Flop Q1: now also RN5.1 (R1)
- net at LD14.1: now also RN7.6 (R3)
- net at LED3.1: now also RN1.6 (R3)
- net Line ~{Y0A}: now reaches IC8.4 (~{Y0A}), IC9.12 (4A)
- net Line ~{Y1A}: now reaches IC8.5 (~{Y1A}), IC9.9 (3A)
- net Line ~{Y2A}: now reaches IC8.6 (~{Y2A}), IC9.5 (2A)
- net Line ~{Y3A}: now reaches IC8.7 (~{Y3A}), IC9.2 (1A)
- net at LED4.1: now also RN1.5 (R4)
- net at LD15.1: now also RN7.5 (R4)
- net at LED2.1: now also RN1.7 (R2)
- net ~{Shift QG}: now reaches IC4.2 (1Y), IC6.2 (1CLR)
- net ~{Shift QH}: now reaches IC4.4 (2Y), IC6.12 (2CLR)
- net at LED7.1: now also RN2.6 (R3)
- net at LED6.1: now also RN2.7 (R2)
- net Count 2QB: now reaches IC6.10 (2QB)
- net Count 2QB: now also RN6.3 (R3)
- net Drive1 4Y: now reaches IC9.11 (4Y)
- net Drive1 4Y: now also RN4.4 (R4)
- net Drive1 1Y: now reaches IC9.3 (1Y)
- net Drive1 1Y: now also RN4.1 (R1)
- net Drive1 2Y: now reaches IC9.6 (2Y)
- net Drive1 2Y: now also RN4.2 (R2)
- net Drive1 3Y: now reaches IC9.8 (3Y)
- net Drive1 3Y: now also RN4.3 (R3)
- net Count 1QA: now reaches IC6.3 (1QA)
- net Count 1QA: now also RN6.2 (R2)
- net at LED1.1: now also RN1.8 (R1)
- new net: LED9.1, RN3.5 (R4)
- new net: IC7.18 (B1), LED9.2
- new net: LD10.1, RN3.6 (R3)
- new net: IC7.17 (B2), LD10.2
- new net: J10.2 (Pin_2), J7.2 (Pin_2)
- new net: IC7.15 (B4), LD12.2
- new net: IC7.16 (B3), LD11.2
- new net: LD12.1, RN3.8 (R1)
- new net: J1.2 (Pin_2), J4.2 (Pin_2)
- new net: LD11.1, RN3.7 (R2)
- new net: J12.2 (Pin_2), J9.2 (Pin_2)
- new net Flop ~{Q2}: IC3.8 (~{Q2}), RN5.4 (R4)
- new net ~{RST}: IC1.1 (~{RST}), IC2.10 (~{SCLR}), IC2.14 (SI), IC4.5 (3A)
- no-connect marks 15 -> 20
Other:
- note added: "Connectors"
- note added: "Power"
- moved on the sheet: C1, C10, C11, C12, C13, C14, C2, C3, C4, C5, C6, C7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

Commit message: Re-re-routed the Clock PCB.
Parts:
- C1, C10, C11, C12, C13, C14, C2, C3, C4, C5, C6, C7, C8, C9: footprint (none) -> Capacitor_SMD:C_0805_2012Metric
- J1, J10, J12, J3, J4, J6, J7, J9: footprint (none) -> Connector_PinHeader_2.54mm:PinHeader_1x02_P2.54mm_Vertical
- J11, J8: footprint (none) -> Connector_PinHeader_2.54mm:PinHeader_1x12_P2.54mm_Vertical
- J2, J5: footprint (none) -> Connector_PinHeader_2.54mm:PinHeader_1x04_P2.54mm_Vertical
- NT1, NT2: footprint (none) -> NetTie:NetTie-2_SMD_Pad0.5mm
- R1, R10, R5: footprint (none) -> Resistor_SMD:R_0805_2012Metric
Connections:
- net at LED9.1: now also RN3.8 (R1); no longer RN3.5 (R4)
- net at LD10.1: now also RN3.7 (R2); no longer RN3.6 (R3)
- net at LD12.1: now also RN3.5 (R4); no longer RN3.8 (R1)
- net at LD11.1: now also RN3.6 (R3); no longer RN3.7 (R2)
Other:
- moved on the sheet: RN3

Commit message: Cleaned up silkscreen.
Parts:
- added NT3: NetTie_2, NetTie:NetTie-2_SMD_Pad0.5mm, symbol Device:NetTie_2
Connections:
- net GND: now also NT3.2; no longer NT1.2
- net Reset Switch: now also NT1.1
- net ~{RST}: now also NT1.2
- net ~{Reset} GND: now also NT3.1; no longer NT1.1
Other:
- note added: "LED Display"
- moved on the sheet: C10, C11, C12, C13, C14, C4, C5, C6, C7, C8, C9, IC1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
