File: Kicad/Computer/VIA Device/W65C22 Breakout Board.kicad_sch (KiCad schematic)
At the start: 13 parts, among them IC1 W65C22S6TQG-14, IC2 AP7365-33WG-7, IC2 W65C22S6TQG-14, IC3 74LVC1G04GV,125, IC6 74LVC1G08GV,125, J12 Conn_01x32_Pin

Commit message: Added an LCD display to the VIA device.
Parts:
- IC1, IC2: Silkscreen (none) -> W65C22S
Changed lines of the file:
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@@
       (effects (font (size 1.27 1.27)) (justify left) hide)
+    )
+    (property "Silkscreen" "W65C22S" (at 201.295 93.345 0)
+      (effects (font (size 1.27 1.27)) hide)
     )
     (pin "1")
@@
       (effects (font (size 1.27 1.27)) (justify left) hide)
     )
-    (pin "1")
+    (property "Silkscreen" "W65C22S" (at 201.295 172.085 0)
+      (effects (font (size 1.27 1.27)) hide)
+    )
+    (pin "1")
