File: Kicad/Desk Lamp/Desk Lamp.kicad_pcb (KiCad board)
At the start: 2 copper layers, 57.5 x 32 mm, 15 parts, among them IC1 LD1117S33C, IC2 MCP73811T-420I/OT, J2 USB-B-S-F-B-TH-R, J5 Conn_01x02_Pin

Commit message: Trying out the Paneliser again.
Parts:
- moved J2 100.9 mm to (117.7, 89.0), turned to 90 degrees
- moved J5 92.5 mm to (111.7, 91.5), turned to 180 degrees
- moved J_{VIN}1 50.1 mm to (86.9, 102.0)
- moved R1 50.1 mm to (87.8, 108.2)
- moved R2 50.1 mm to (87.8, 110.5)
- moved IC1 50.1 mm to (94.1, 97.3)
- moved LED1 50.1 mm to (94.1, 106.8)
- moved J_{Switch}1 49.9 mm to (127.7, 106.1)
- moved C1 49.6 mm to (118.3, 118.5)
- moved C2 49.6 mm to (126.3, 118.5)
- moved H1 49.6 mm to (122.4, 112.1)
- moved IC2 49.6 mm to (122.0, 119.4)
- moved J_{Battery+}1 49.6 mm to (129.3, 114.9)
- moved J_{VUSB+}1 49.6 mm to (115.2, 114.7)
- moved J_{VOUT}1 49.4 mm to (117.0, 106.1)
Routing:
- net /GND: track 32.4 -> 44.3 mm
- net Net-(J2-GND): track 0.00 -> 9.30 mm
- net Net-(J2-VBUS): track 0.00 -> 7.06 mm
- net /5V: track 11.8 -> 14.3 mm
- net /3.7V: track 16.0 -> 16.8 mm
Other:
- board size 57.5 x 32 mm -> 55.2 x 41.4 mm
