File: Kicad/Computer/Video/Video Board/Video Board.kicad_sch (KiCad schematic)
At the start: 48 parts, among them IC1 74LVC2G04GW-Q100H, IC1 LD1117S50C, IC100 74LVC1G157GV,125, IC101 74LVC1G157GV,125, IC13 74LVC574APW,118, IC2 SST39VF010-70-4I-NHE, IC27 74LVC1GX04GW,125, J5 395-098-520-350

Commit message: Added Video Signals and Video Memory.
Parts:
- removed C23 (x3): 1μF, SamacSys_Parts:C_0805, symbol HCP65:C_0805
- removed IC100, IC101: 74LVC1G157GV,125, 74LVC1G157GV125, symbol Nexperia:74LVC1G157GV,125
- removed IC13: 74LVC574APW,118, SOP65P640X110-20N, symbol Nexperia:74LVC574APW,118
- added B26: Video Signals Output, HCP65_Parts:HCP65_Video_Output_Signals, symbol HCP65:Video_Signals_Output
- added B27: Counter 24bit with IO, HCP65_Parts:HCP65_Counter_24bit_with_IO, symbol HCP65:Counter_24bit_with_IO
- added B28: Memory 32KB, HCP65_Parts:HCP65_Memory_32KB_With_Latch, symbol HCP65:Memory_32KB
- added B29, B30: Selector 12bit, HCP65_Parts:HCP65_Selector_12bit, symbol HCP65:Selector_12bit
- added IC10: 74LVC04APW,118, SOP65P640X110-14N, symbol Nexperia:74LVC04APW,118
- added IC11, IC7: SN74CBT3257CPWR, SOP65P640X120-16N, symbol Texas_Instruments:SN74CBT3257CPWR
- added IC3, IC6: IS61WV20488FBLL-10TLI, SOP80P1176X120-44N, symbol ISSI:IS61WV20488FBLL-10TLI
- added IC8: 74LVC161PW,112, SOP65P640X110-16N, symbol Nexperia:74LVC161PW,112
- added IC9: 74LVC138APW-Q100J, SOP65P640X110-16N, symbol Nexperia:74LVC138APW-Q100J
- B24: footprint (none) -> HCP65_Parts:HCP65_D_Flip_Flop
- B8: value Flags Interrupt -> Flags & Interrupt; Silkscreen Flags Interrupt -> Flags & Interrupt
- C12: footprint (none) -> Capacitor_THT:CP_Radial_D4.0mm_P2.00mm
- LED1: footprint (none) -> LED_THT:LED_D5.0mm
Connections:
- net 3.3V: now also B2.19 (IR0), B21.19 (IR0), B30.16 (B10), IC10.14 (3V), IC8.10 (CET), IC8.16 (3V), IC8.9 (~{PE}), IC9.16 (3V), IC9.6 (E3); no longer B2.16 (IR0), B21.16 (IR0)
- net 5V: now also B26.1 (5V), B26.17 (5V), B27.3 (5V), B27.35 (5V), B28.20 (5V), B29.20 (5V), B30.20 (5V)
- net A0: now also B29.14 (A0)
- net A1: now also B29.13 (A1)
- net A10: now also B29.4 (A10)
- net A11: now also B29.3 (A11)
- net A12: now also B30.5 (A9)
- net A13: now also B30.6 (A8)
- net A14: now also B30.7 (A7)
- net A2: now also B29.12 (A2)
- net A3: now also B29.11 (A3)
- net A4: now also B29.10 (A4)
- net A5: now also B29.9 (A5)
- net A6: now also B29.8 (A6)
- net A7: now also B29.7 (A7)
- net A8: now also B29.6 (A8)
- net A9: now also B29.5 (A9)
- net Advance Pixel: now also B18.36 (Count_Enable), B27.29 (Count_Enable); no longer B18.64 (Count_Enable)
- net C0: now also B18.37 (C0), B27.37 (C0); no longer B18.59 (C0)
- net C1: now also B18.38 (C1), B27.38 (C1); no longer B18.58 (C1)
- net C10: now also B27.48 (C10)
- net C11: now also B18.49 (C11), B27.49 (C11); no longer B18.47 (C11)
- net C12: now also B18.50 (C12), B27.50 (C12); no longer B18.46 (C12)
- net C13: now also B18.51 (C13), B27.51 (C13); no longer B18.45 (C13)
- net C14: now also B18.52 (C14), B27.52 (C14); no longer B18.44 (C14)
- net C15: now also B18.53 (C15), B27.53 (C15); no longer B18.43 (C15)
- net C16: now also B18.54 (C16), B27.54 (C16); no longer B18.41 (C16)
- net C17: now also B18.56 (C17), B27.56 (C17); no longer B18.40 (C17)
- net C18: now also B18.57 (C18), B27.57 (C18); no longer B18.39 (C18)
- net C19: now also B18.58 (C19), B27.58 (C19); no longer B18.38 (C19)
- net C2: now also B18.39 (C2), B27.39 (C2); no longer B18.57 (C2)
- net C20: now also B18.59 (C20), B27.59 (C20); no longer B18.37 (C20)
- net C3: now also B18.40 (C3), B27.40 (C3); no longer B18.56 (C3)
- net C4: now also B18.41 (C4), B27.41 (C4); no longer B18.54 (C4)
- net C5: now also B18.43 (C5), B27.43 (C5); no longer B18.53 (C5)
- net C6: now also B18.44 (C6), B27.44 (C6); no longer B18.52 (C6)
- net C7: now also B18.45 (C7), B27.45 (C7); no longer B18.51 (C7)
- net C8: now also B18.46 (C8), B27.46 (C8); no longer B18.50 (C8)
- net C9: now also B18.47 (C9), B27.47 (C9); no longer B18.49 (C9)
- net D0: now also B27.17 (D7), B28.39 (D7)
- net D1: now also B27.18 (D6), B28.38 (D6)
- net D2: now also B27.19 (D5), B28.37 (D5)
- net D3: now also B27.20 (D4), B28.36 (D4)
- net D4: now also B27.21 (D3), B28.35 (D3)
- net D5: now also B27.22 (D2), B28.34 (D2)
- net D6: now also B27.24 (D1), B28.33 (D1)
- net D7: now also B27.25 (D0), B28.32 (D0)
- net First Pixel: now also B21.17 (CLK), B26.9 (First_Pixel); no longer B21.19 (CLK)
- net First Pixel _{HALF CYCLE}: now also B26.24 (First_Pixel_{OUT}), IC8.2 (CP)
- net First Row: now also B26.11 (First_Row)
- net First Row _{HALF CYCLE}: now also B26.22 (First_Row_{OUT})
- net GND: now also B18.2 (L23), B18.4 (L22), B18.5 (L21), B2.20 (IR1), B21.20 (IR1), B26.12 (GND), B26.21 (GND), B26.28 (GND), B26.5 (GND), B27.10 (GND), B27.23 (GND), B27.42 (GND), B27.55 (GND), B28.21 (GND), B28.40 (GND), B29.1 (~{E}), B29.40 (GND), B30.1 (~{E}), B30.15 (B11), B30.17 (B9), B30.18 (B8), B30.19 (B7), B30.40 (GND), IC10.11 (5A), IC10.13 (6A), IC10.7 (GND), IC8.3 (D0), IC8.4 (D1), IC8.5 (D2), IC8.6 (D3), IC8.8 (GND), IC9.4 (~{E1}), IC9.5 (~{E2}), IC9.8 (GND); no longer B2.17 (IR1), B21.17 (IR1)
- net H10: now also B2.37 (R10); no longer B2.26 (R10)
- net H3: now also B2.29 (R3); no longer B2.35 (R3)
- net H4: now also B2.30 (R4); no longer B2.33 (R4)
- net H5: now also B2.31 (R5); no longer B2.32 (R5)
- net H6: now also B2.32 (R6); no longer B2.31 (R6)
- net H7: now also B2.33 (R7); no longer B2.30 (R7)
- net H8: now also B2.35 (R8); no longer B2.29 (R8)
- net H9: now also B2.36 (R9); no longer B2.28 (R9)
- net Horizontal Blank: now also B18.29 (~{Latch_Count}), B26.7 (Horizontal_Blank), B27.9 (~{Load_Count_Start}); no longer B18.2 (~{Latch_Count})
- net Horizontal Blank _{HALF CYCLE}: now also B26.27 (Horizontal_Blank_{OUT})
- net Horizontal Sync: now also B26.4 (Horizontal_Sync)
- net Horizontal Sync Polarity: now also B26.3 (Horizontal_Sync_Polarity)
- net Horizontal Sync _{HALF CYCLE}: now also B26.29 (Horizontal_Sync_{OUT})
- net L0: now also B18.28 (L0); no longer B18.4 (L0)
- net L1: now also B18.27 (L1); no longer B18.5 (L1)
- net L10: now also B18.17 (L10); no longer B18.15 (L10)
- net L11: now also B18.16 (L11); no longer B18.18 (L11)
- net L12: now also B18.15 (L12); no longer B18.19 (L12)
- net L13: now also B18.14 (L13); no longer B18.20 (L13)
- net L14: now also B18.13 (L14); no longer B18.21 (L14)
- net L15: now also B18.12 (L15); no longer B18.22 (L15)
- net L16: now also B18.11 (L16); no longer B18.24 (L16)
- net L17: now also B18.9 (L17); no longer B18.25 (L17)
- net L18: now also B18.8 (L18); no longer B18.26 (L18)
- net L19: now also B18.7 (L19); no longer B18.27 (L19)
- net L2: now also B18.26 (L2); no longer B18.6 (L2)
- net L20: now also B18.6 (L20); no longer B18.28 (L20)
- net L3: now also B18.25 (L3); no longer B18.7 (L3)
- net L4: now also B18.24 (L4); no longer B18.8 (L4)
- net L5: now also B18.22 (L5); no longer B18.9 (L5)
- net L6: now also B18.21 (L6); no longer B18.11 (L6)
- net L7: now also B18.20 (L7); no longer B18.12 (L7)
- net L8: now also B18.19 (L8); no longer B18.13 (L8)
- net L9: now also B18.18 (L9); no longer B18.14 (L9)
- net Last Pixel + 1: now also B26.10 (Last_Pixel+1)
- net Last Pixel + 1 _{HALF CYCLE}: now also B26.23 (Last_Pixel+1_{OUT})
- net Last Row + 1: now also B26.13 (Last_Row+1)
- net Last Row + 1 _{HALF CYCLE}: now also B26.20 (Last_Row+1_{OUT})
- net Latch Address Bank: now also B18.32 (Latch_Bank); no longer B18.31 (Latch_Bank)
- net Latch Address High: now also B18.31 (Latch_High); no longer B18.30 (Latch_High)
- net Latch Address Low: now also B18.30 (Latch_Low); no longer B18.29 (Latch_Low)
- net Pixel CLK: now also B18.64 (Pixel_CLK), B2.17 (CLK), B27.8 (CLK); no longer B18.16 (Pixel_CLK), B2.19 (CLK)
- net R0: now also B21.25 (R0), B29.27 (B0); no longer B21.38 (R0)
- net R1: now also B21.26 (R1), B29.26 (B1); no longer B21.37 (R1)
- net R2: now also B21.28 (R2), B29.25 (B2); no longer B21.36 (R2)
- net R3: now also B21.29 (R3), B29.24 (B3); no longer B21.35 (R3)
- net R4: now also B21.30 (R4), B29.23 (B4); no longer B21.33 (R4)
- net R5: now also B21.31 (R5), B29.22 (B5); no longer B21.32 (R5)
- net R6: now also B21.32 (R6), B29.21 (B6); no longer B21.31 (R6)
- net R7: now also B21.33 (R7), B29.19 (B7); no longer B21.30 (R7)
- net R8: now also B21.35 (R8), B29.18 (B8); no longer B21.29 (R8)
- net R9: now also B21.36 (R9), B29.17 (B9); no longer B21.28 (R9)
- net Read Address Bank: now also B27.1 (Read_Count_Bank)
- net Read Address High: now also B27.2 (Read_Count_High)
- net Read Address Low: now also B27.4 (Read_Count_Low), B27.5 (Enable_Latch_Read_Count)
- net Vertical Blank: now also B26.8 (Vertical_Blank)
- net Vertical Blank _{HALF CYCLE}: now also B26.25 (Vertical_Blank_{OUT})
- net Vertical Sync: now also B26.15 (Vertical_Sync)
- net Vertical Sync Polarity: now also B26.14 (Vertical_Sync_Polarity)
- net Vertical Sync _{HALF CYCLE}: now also B26.26 (Vertical_Sync_{OUT})
- net ~{Device RAM}: now also B29.2 (S), B30.2 (S)
- net ~{Horizontal Sync}: now also B26.6 (~{Horizontal_Sync})
- net ~{Pixel CLK}: now also B26.2 (~{Pixel_CLK}); no longer B18.17 (~{Pixel_CLK})
- net ~{RD}: now also B30.3 (A11)
- net ~{Reset}: now also B27.13 (~{Reset})
- net ~{Vertical Blank}: now also IC8.1 (~{MR})
- net ~{Vertical Sync}: now also B26.16 (~{Vertical_Sync})
- net ~{WD}: now also B28.2 (T~{DIR}), B30.4 (A10)
- new net LA0: B29.16 (B10), IC8.14 (Q0), IC9.1 (A0)
- new net LA1: B29.15 (B11), IC8.13 (Q1), IC9.2 (A1)
- new net LA2: IC8.12 (Q2), IC8.7 (CEP), IC9.3 (A2)
- new net Latch Loaded Address: IC10.8 (4Y)
- new net Load Address Bank: B27.30 (Write_Start_Bank), IC10.6 (3Y)
- new net Load Address High: B27.31 (Write_Start_High), IC10.4 (2Y)
- new net Load Address Low: B27.32 (Write_Start_Low), IC10.2 (1Y)
- new net RA0: B28.19 (M0), B29.28 (Q0)
- new net RA1: B28.18 (M1), B29.29 (Q1)
- new net RA10: B28.9 (M10), B29.38 (Q10)
- new net RA11: B28.8 (M11), B29.39 (Q11)
- new net RA12: B28.7 (M12), B30.35 (Q7)
- new net RA13: B28.6 (M13), B30.36 (Q8)
- new net RA14: B28.5 (M14), B30.37 (Q9)
- new net RA2: B28.17 (M2), B29.30 (Q2)
- new net RA3: B28.16 (M3), B29.31 (Q3)
- new net RA4: B28.15 (M4), B29.32 (Q4)
- new net RA5: B28.14 (M5), B29.33 (Q5)
- new net RA6: B28.13 (M6), B29.34 (Q6)
- new net RA7: B28.12 (M7), B29.35 (Q7)
- new net RA8: B28.11 (M8), B29.36 (Q8)
- new net RA9: B28.10 (M9), B29.37 (Q9)
- new net Row Address ~{OE}: B28.3 (M~{OE}), B30.39 (Q11)
- new net Row Address ~{OE}·~{WE}: B28.1 (T~{OE})
- new net Row Address ~{WE}: B28.4 (M~{WE}), B30.38 (Q10)
- new net ~{Latch Loaded Address}: IC10.9 (4A), IC9.12 (~{Y3})
- new net ~{Load Address Bank}: IC10.5 (3A), IC9.13 (~{Y2})
- new net ~{Load Address High}: IC10.3 (2A), IC9.14 (~{Y1})
- new net ~{Load Address Low}: IC10.1 (1A), IC9.15 (~{Y0})
- no-connect marks 78 -> 93
Other:
- moved on the sheet: B1, B10, B11, B15, B16, B19, B23, B24, B25, B4, B8, B9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

Commit message: Added Video Memory 2MB and D-type Flip Flop 16bit.
Parts:
- removed B17: Comparator 10bit, HCP65_Parts:HCP65_Comparator_10bit, symbol HCP65:Comparator_10bit
- removed B18: Video Address Counter, HCP65_Parts:HCP65_Video_Address_Counter, symbol HCP65:Video_Address_Counter
- removed B19: Video Address Reader, HCP65_Parts:HCP65_Video_Address_Reader, symbol HCP65:Video_Address_Reader
- removed B22: Video Pixel Doubler, HCP65_Parts:HCP65_Video_Pixel_Doubler, symbol HCP65:Video_Pixel_Doubler
- removed B27: Counter 24bit with IO, HCP65_Parts:HCP65_Counter_24bit_with_IO, symbol HCP65:Counter_24bit_with_IO
- removed B4: Video Address Selector, HCP65_Parts:HCP65_Video_Address_Selector, symbol HCP65:Video_Address_Selector
- removed IC10: 74LVC04APW,118, SOP65P640X110-14N, symbol Nexperia:74LVC04APW,118
- removed IC11, IC7: SN74CBT3257CPWR, SOP65P640X120-16N, symbol Texas_Instruments:SN74CBT3257CPWR
- removed IC3, IC6: IS61WV20488FBLL-10TLI, SOP80P1176X120-44N, symbol ISSI:IS61WV20488FBLL-10TLI
- removed IC8: 74LVC161PW,112, SOP65P640X110-16N, symbol Nexperia:74LVC161PW,112
- added B17: Video Address Reader, HCP65_Parts:HCP65_Video_Address_Reader, symbol HCP65:Video_Address_Reader
- added B18, B31, B32, B4: Video Memory 2MB, HCP65_Parts:HCP65_Video_Memory_2MB, symbol HCP65:Video_Memory_2MB
- added B19: D-type Flip Flop 16bit, HCP65_Parts:HCP65_D_Flip_Flop_16bit, symbol HCP65:D_Flip_Flop_16bit
- added B22: Video Address Counter, HCP65_Parts:HCP65_Video_Address_Counter, symbol HCP65:Video_Address_Counter
- added IC10: 74LVC32APW,118, SOP65P640X110-14N, symbol Nexperia:74LVC32APW,118
- added IC11, IC12, IC13, IC14: 74LVC574APW,118, SOP65P640X110-20N, symbol Nexperia:74LVC574APW,118
- added IC3, IC7: 74LVC08APW,112, SOP65P640X110-14N, symbol Nexperia:74LVC08APW,112
- added IC6: 74LVC04APW,118, SOP65P640X110-14N, symbol Nexperia:74LVC04APW,118
- added IC8: 74LVC163PW,118, SOP65P640X110-16N, symbol Nexperia:74LVC163PW,118
Connections:
- net Video Address ~{OE} is gone; now on net GND: B24.1 (~{OE})
- net ~{CPU Address} is gone; now on net ~{Device RAM}: B11.23 (~{Device_RAM})
- net ~{Latch Loaded Address} is gone; now on net ~{Load Address Bank}: IC9.12 (~{Y3})
- net ~{Vertical Interrupt} _{CMP} is gone; now on net ~{Vertical Blank}: B8.4 (~{Set_Interrupt_on_CLK})
- net 3.3V: now also B28.22 (LLE), B18.69 (V~{WE}), B31.69 (V~{WE}), B32.69 (V~{WE}), B4.69 (V~{WE}), IC11.20 (3V), IC12.20 (3V), IC13.20 (3V), IC14.20 (3V), IC3.14 (3V), IC6.14 (3V), IC8.10 (CET)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
- net 5V: now also B17.23 (5V), B17.3 (5V), B18.3 (5V), B18.39 (5V), B19.23 (5V), B19.3 (5V), B22.3 (5V), B22.31 (5V), B31.3 (5V), B31.39 (5V), B32.3 (5V), B32.39 (5V)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
- net A0_{M}: now also B18.28 (MA0), B31.28 (MA0), B32.28 (MA0), B4.28 (MA0)
- net A10_{M}: now also B18.17 (MA10), B31.17 (MA10), B32.17 (MA10), B4.17 (MA10)
- net A11_{M}: now also B18.16 (MA11), B31.16 (MA11), B32.16 (MA11), B4.16 (MA11)
- net A12: now also B30.10 (A4); no longer B30.5 (A9)
- net A12_{M}: now also B18.15 (MA12), B31.15 (MA12), B32.15 (MA12), B4.15 (MA12)
- net A13: now also B30.9 (A5); no longer B30.6 (A8)
- net A13_{M}: now also B18.14 (MA13), B31.14 (MA13), B32.14 (MA13), B4.14 (MA13)
- net A14: now also B30.8 (A6); no longer B30.7 (A7)
- net A14_{M}: now also B18.13 (MA14), B31.13 (MA14), B32.13 (MA14), B4.13 (MA14)
- net A15: now also B30.7 (A7)
- net A15_{M}: now also B18.12 (MA15), B31.12 (MA15), B32.12 (MA15), B4.12 (MA15)
- net A16: now also B30.6 (A8)
- net A16_{M}: now also B18.11 (MA16), B31.11 (MA16), B32.11 (MA16), B4.11 (MA16)
- net A17_{M}: now also B18.9 (MA17), B31.9 (MA17), B32.9 (MA17), B4.9 (MA17)
- net A18_{M}: now also B18.8 (MA18), B31.8 (MA18), B32.8 (MA18), B4.8 (MA18)
- net A19_{M}: now also B18.7 (MA19), B31.7 (MA19), B32.7 (MA19), B4.7 (MA19)
- net A1_{M}: now also B18.26 (MA1), B31.26 (MA1), B32.26 (MA1), B4.26 (MA1)
- net A20_{M}: now also B18.6 (MA20), B31.6 (MA20), B32.6 (MA20), B4.6 (MA20)
- net A2_{M}: now also B18.25 (MA2), B31.25 (MA2), B32.25 (MA2), B4.25 (MA2)
- net A3_{M}: now also B18.23 (MA4), B31.23 (MA4), B32.23 (MA4), B4.23 (MA4)
- net A4_{M}: now also B18.24 (MA3), B31.24 (MA3), B32.24 (MA3), B4.24 (MA3)
- net A5_{M}: now also B18.22 (MA5), B31.22 (MA5), B32.22 (MA5), B4.22 (MA5)
- net A6_{M}: now also B18.21 (MA6), B31.21 (MA6), B32.21 (MA6), B4.21 (MA6)
- net A7_{M}: now also B18.20 (MA7), B31.20 (MA7), B32.20 (MA7), B4.20 (MA7)
- net A8_{M}: now also B18.19 (MA8), B31.19 (MA8), B32.19 (MA8), B4.19 (MA8)
- net A9_{M}: now also B18.18 (MA9), B31.18 (MA9), B32.18 (MA9), B4.18 (MA9)
- net Advance Pixel: now also B22.26 (Count_Enable)
- net C0: now also B17.21 (C0), B22.30 (C0)
- net C1: now also B17.22 (C1), B22.32 (C1)
- net C10: now also B17.18 (C10), B22.42 (C10)
- net C11: now also B17.17 (C11), B22.43 (C11)
- net C12: now also B17.16 (C12), B22.44 (C12)
- net C13: now also B17.15 (C13), B22.45 (C13)
- net C14: now also B17.13 (C14), B22.46 (C14)
- net C15: now also B17.12 (C15), B22.48 (C15)
- net C16: now also B17.11 (C16), B22.49 (C16)
- net C17: now also B17.10 (C17), B22.50 (C17)
- net C18: now also B17.9 (C18), B22.51 (C18)
- net C19: now also B17.8 (C19), B22.52 (C19)
- net C2: now also B17.24 (C2), B22.33 (C2)
- net C20: now also B17.5 (C20), B22.53 (C20)
- net C3: now also B17.25 (C3), B22.34 (C3)
- net C4: now also B17.26 (C4), B22.35 (C4)
- net C5: now also B17.28 (C5), B22.36 (C5)
- net C6: now also B17.29 (C6), B22.38 (C6)
- net C7: now also B17.30 (C7), B22.39 (C7)
- net C8: now also B17.20 (C8), B22.40 (C8)
- net C9: now also B17.19 (C9), B22.41 (C9)
- net D0: now also B17.31 (D0)
- net D0_{M}: now also B18.36 (MD0), B31.36 (MD0), B32.36 (MD0), B4.36 (MD0)
- net D1: now also B17.32 (D1)
- net D1_{M}: now also B18.35 (MD1), B31.35 (MD1), B32.35 (MD1), B4.35 (MD1)
- net D2: now also B17.33 (D2)
- net D2_{M}: now also B18.34 (MD2), B31.34 (MD2), B32.34 (MD2), B4.34 (MD2)
- net D3: now also B17.35 (D3)
- net D3_{M}: now also B18.33 (MD3), B31.33 (MD3), B32.33 (MD3), B4.33 (MD3)
- net D4: now also B17.36 (D4)
- net D4_{M}: now also B18.32 (MD4), B31.32 (MD4), B32.32 (MD4), B4.32 (MD4)
- net D5: now also B17.37 (D5)
- net D5_{M}: now also B18.31 (MD5), B31.31 (MD5), B32.31 (MD5), B4.31 (MD5)
- net D6: now also B17.38 (D6)
- net D6_{M}: now also B18.30 (MD6), B31.30 (MD6), B32.30 (MD6), B4.30 (MD6)
- net D7: now also B17.39 (D7)
- net D7_{M}: now also B18.29 (MD7), B31.29 (MD7), B32.29 (MD7), B4.29 (MD7)
- net First Pixel _{HALF CYCLE}: now also IC11.9 (D7), IC8.2 (CP)
- net First Row _{HALF CYCLE}: now also IC11.7 (D5)
- net GND: now also B28.23 (L~{OE}), B30.11 (A3), B30.12 (A2), B30.13 (A1), B30.14 (A0), B30.21 (B6), B30.22 (B5), B30.23 (B4), B30.24 (B3), B30.25 (B2), B30.26 (B1), B30.27 (B0)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
- net Horizontal Blank _{HALF CYCLE}: now also IC11.4 (D2)
- net Horizontal Sync _{HALF CYCLE}: now also IC11.5 (D3)
- net LA0: now also B29.27 (B0), IC8.14 (Q0); no longer B29.16 (B10)
- net LA1: now also B29.26 (B1), IC8.13 (Q1); no longer B29.15 (B11)
- net LA2: now also IC8.12 (Q2)
- net Last Pixel + 1 _{HALF CYCLE}: now also IC11.8 (D6)
- net Last Row + 1 _{HALF CYCLE}: now also IC11.6 (D4)
- net Pixel CLK: now also B22.4 (CLK), IC11.11 (CP), IC13.11 (CP)
- net RA12: now also B30.32 (Q4); no longer B30.35 (Q7)
- net RA13: now also B30.33 (Q5); no longer B30.36 (Q8)
- net RA14: now also B30.34 (Q6); no longer B30.37 (Q9)
- net Read Address Bank: now also B17.1 (Read_Address_Bank)
- net Read Address High: now also B17.2 (Read_Address_High)
- net Read Address Low: now also B17.4 (Read_Address_Low)
- net VA0: now also B18.47 (VA0), B31.47 (VA0), B32.47 (VA0), B4.47 (VA0)
- net VA1: now also B18.48 (VA1), B31.48 (VA1), B32.48 (VA1), B4.48 (VA1)
- net VA10: now also B18.57 (VA10), B31.57 (VA10), B32.57 (VA10), B4.57 (VA10)
- net VA11: now also B18.58 (VA11), B31.58 (VA11), B32.58 (VA11), B4.58 (VA11)
- net VA12: now also B18.59 (VA12), B31.59 (VA12), B32.59 (VA12), B4.59 (VA12)
- net VA13: now also B18.60 (VA13), B31.60 (VA13), B32.60 (VA13), B4.60 (VA13)
- net VA14: now also B18.61 (VA14), B31.61 (VA14), B32.61 (VA14), B4.61 (VA14)
- net VA15: now also B18.62 (VA15), B31.62 (VA15), B32.62 (VA15), B4.62 (VA15)
- net VA16: now also B18.64 (VA16), B31.64 (VA16), B32.64 (VA16), B4.64 (VA16)
- net VA17: now also B18.65 (VA17), B31.65 (VA17), B32.65 (VA17), B4.65 (VA17)
- net VA18: now also B18.66 (VA18), B31.66 (VA18), B32.66 (VA18), B4.66 (VA18)
- net R0 renamed Row0
- net R1 renamed Row1
- net R2 renamed Row2
- net R3 renamed Row3
- net R4 renamed Row4
- net R5 renamed Row5
- net R6 renamed Row6
- net R7 renamed Row7
- net R8 renamed Row8
- net R9 renamed Row9
- net Row Address ~{OE}·~{WE} renamed (~{RD}·~{WD})+~{Device RAM}
- new net A17: B30.5 (A9)
- new net D~{OE}G0: B32.72 (D~{OE}), IC3.3 (1Y)
- new net D~{OE}G1: B4.72 (D~{OE}), IC3.8 (3Y)
- new net D~{OE}P0: B31.72 (D~{OE}), IC3.6 (2Y)
- new net D~{OE}P1: B18.72 (D~{OE}), IC3.11 (4Y)
- new net First Pixel _{CYCLE 1H}: IC11.12 (Q7), IC12.9 (D7)
- new net First Pixel _{CYCLE 1}: IC12.12 (Q7), IC13.9 (D7)
- new net First Pixel _{CYCLE 2H}: IC13.12 (Q7), IC14.9 (D7)
- new net First Pixel _{CYCLE 2}: IC14.12 (Q7)
- new net First Row _{CYCLE 1H}: IC11.14 (Q5), IC12.7 (D5)
- new net First Row _{CYCLE 1}: IC12.14 (Q5), IC13.7 (D5)
- new net First Row _{CYCLE 2H}: IC13.14 (Q5), IC14.7 (D5)
- new net First Row _{CYCLE 2}: IC14.14 (Q5)
- new net Horizontal Blank _{CYCLE 1H}: IC11.17 (Q2), IC12.4 (D2)
- new net Horizontal Blank _{CYCLE 1}: IC12.17 (Q2), IC13.4 (D2)
- new net Horizontal Blank _{CYCLE 2H}: IC13.17 (Q2), IC14.4 (D2)
- new net Horizontal Blank _{CYCLE 2}: IC14.17 (Q2)
- new net Horizontal Sync _{CYCLE 1H}: IC11.16 (Q3), IC12.5 (D3)
- new net Horizontal Sync _{CYCLE 1}: IC12.16 (Q3), IC13.5 (D3)
- new net Horizontal Sync _{CYCLE 2H}: IC13.16 (Q3), IC14.5 (D3)
- new net Horizontal Sync _{CYCLE 2}: IC14.16 (Q3)
- new net Last Pixel + 1 _{CYCLE 1H}: IC11.13 (Q6), IC12.8 (D6)
- new net Last Pixel + 1 _{CYCLE 1}: IC12.13 (Q6), IC13.8 (D6)
- new net Last Pixel + 1 _{CYCLE 2H}: IC13.13 (Q6), IC14.8 (D6)
- new net Last Pixel + 1 _{CYCLE 2}: IC14.13 (Q6)
- new net Last Row + 1 _{CYCLE 1H}: IC11.15 (Q4), IC12.6 (D4)
- new net Last Row + 1 _{CYCLE 1}: IC12.15 (Q4), IC13.6 (D4)
- new net Last Row + 1 _{CYCLE 2H}: IC13.15 (Q4), IC14.6 (D4)
- new net Last Row + 1 _{CYCLE 2}: IC14.15 (Q4)
- new net VGD0: B19.11 (IN8), B32.37 (VD0), B4.37 (VD0)
- new net VGD0 _{CYCLE 2}: B19.31 (OUT8)
- new net VGD1: B19.10 (IN9), B32.38 (VD1), B4.38 (VD1)
- new net VGD1 _{CYCLE 2}: B19.32 (OUT9)
- new net VGD2: B19.9 (IN10), B32.40 (VD2), B4.40 (VD2)
- new net VGD2 _{CYCLE 2}: B19.33 (OUT10)
- new net VGD3: B19.8 (IN11), B32.41 (VD3), B4.41 (VD3)
- new net VGD3 _{CYCLE 2}: B19.35 (OUT11)
- new net VGD4: B19.6 (IN12), B32.42 (VD4), B4.42 (VD4)
- new net VGD4 _{CYCLE 2}: B19.36 (OUT12)
- new net VGD5: B19.5 (IN13), B32.43 (VD5), B4.43 (VD5)
- new net VGD5 _{CYCLE 2}: B19.37 (OUT13)
- new net VGD6: B19.4 (IN14), B32.44 (VD6), B4.44 (VD6)
- new net VGD6 _{CYCLE 2}: B19.38 (OUT14)
- new net VGD7: B19.2 (IN15), B32.45 (VD7), B4.45 (VD7)
- new net VGD7 _{CYCLE 2}: B19.39 (OUT15)
- new net VPD0: B18.37 (VD0), B19.20 (IN0), B31.37 (VD0)
- new net VPD0 _{CYCLE 2}: B19.21 (OUT0)
- new net VPD1: B18.38 (VD1), B19.19 (IN1), B31.38 (VD1)
- new net VPD1 _{CYCLE 2}: B19.22 (OUT1)
- new net VPD2: B18.40 (VD2), B19.18 (IN2), B31.40 (VD2)
- new net VPD2 _{CYCLE 2}: B19.24 (OUT2)
- new net VPD3: B18.41 (VD3), B19.17 (IN3), B31.41 (VD3)
- new net VPD3 _{CYCLE 2}: B19.25 (OUT3)
- new net VPD4: B18.42 (VD4), B19.16 (IN4), B31.42 (VD4)
- new net VPD4 _{CYCLE 2}: B19.26 (OUT4)
- new net VPD5: B18.43 (VD5), B19.15 (IN5), B31.43 (VD5)
- new net VPD5 _{CYCLE 2}: B19.28 (OUT5)
- new net VPD6: B18.44 (VD6), B19.13 (IN6), B31.44 (VD6)
- new net VPD6 _{CYCLE 2}: B19.29 (OUT6)
- new net VPD7: B18.45 (VD7), B19.12 (IN7), B31.45 (VD7)
- new net VPD7 _{CYCLE 2}: B19.30 (OUT7)
- new net Vertical Blank _{CYCLE 1H}: IC11.19 (Q0), IC12.2 (D0)
- new net Vertical Blank _{CYCLE 1}: IC12.19 (Q0), IC13.2 (D0)
- new net Vertical Blank _{CYCLE 2H}: IC13.19 (Q0), IC14.2 (D0)
- new net Vertical Blank _{CYCLE 2}: IC14.19 (Q0)
- new net Vertical Sync _{CYCLE 1H}: IC11.18 (Q1), IC12.3 (D1)
- new net Vertical Sync _{CYCLE 1}: IC12.18 (Q1), IC13.3 (D1)
- new net Vertical Sync _{CYCLE 2H}: IC13.18 (Q1), IC14.3 (D1)
- new net Vertical Sync _{CYCLE 2}: IC14.18 (Q1)
- new net ~{Memory Frame}: B18.1 (D), B4.1 (D), IC3.2 (1B), IC3.5 (2B), IC6.2 (1Y)
- new net ~{RD}·~{WD}: IC10.1 (1A), IC7.3 (1Y)
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Other:
- note added: "Because VA (Video Address) is only latched on ~{Pixel CLK} that means if if VG and VP are also latched on ~{Pixel Clock} then they will still be holding the old values before VA changes."
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
Commit message: Mostly added an 18bit selector.
Parts:
- added B27, B34: Selector 12bit, HCP65_Parts:HCP65_Selector_12bit, symbol HCP65:Selector_12bit
- added B33: Memory 32KB, HCP65_Parts:HCP65_Memory_32KB_With_Latch, symbol HCP65:Memory_32KB
- added IC15: 74LVC138APW-Q100J, SOP65P640X110-16N, symbol Nexperia:74LVC138APW-Q100J
Connections:
- net A17 is gone; now on net A16: B30.5 (A9)
- net (~{RD}·~{WD})+~{Device RAM}: now also B33.1 (T~{OE}); no longer B28.1 (T~{OE}), IC10.3 (1Y)
- net 3.3V: now also B30.21 (B6), IC10.14 (3V), IC7.14 (3V), B33.22 (LLE), B34.16 (B10), IC15.16 (3V), IC15.6 (E3)
- net 5V: now also B27.20 (5V), B33.20 (5V), B34.20 (5V)
- net A0: now also B27.14 (A0)
- net A1: now also B27.13 (A1)
- net A10: now also B27.4 (A10)
- net A11: now also B27.3 (A11)
- net A12: now also B30.9 (A5), B34.9 (A5); no longer B30.10 (A4)
- net A13: now also B30.8 (A6), B34.8 (A6); no longer B30.9 (A5)
- net A14: now also B30.7 (A7), B34.7 (A7), IC15.1 (A0); no longer B30.8 (A6)
- net A15: now also B30.6 (A8), B34.6 (A8), IC15.2 (A1); no longer B30.7 (A7)
- net A16: now also B34.5 (A9), IC15.3 (A2); no longer B30.6 (A8)
- net A2: now also B27.12 (A2)
- net A3: now also B27.11 (A3)
- net A4: now also B27.10 (A4)
- net A5: now also B27.9 (A5)
- net A6: now also B27.8 (A6)
- net A7: now also B27.7 (A7)
- net A8: now also B27.6 (A8)
- net A9: now also B27.5 (A9)
- net D0: now also B33.39 (D7)
- net D1: now also B33.38 (D6)
- net D2: now also B33.37 (D5)
- net D3: now also B33.36 (D4)
- net D4: now also B33.35 (D3)
- net D5: now also B33.34 (D2)
- net D6: now also B33.33 (D1)
- net D7: now also B33.32 (D0)
- net GND: now also B30.10 (A4), IC10.7 (GND), IC7.7 (GND), B27.1 (~{E}), B27.40 (GND), B33.21 (GND), B33.23 (L~{OE}), B33.40 (GND), B34.1 (~{E}), B34.10 (A4), B34.11 (A3), B34.12 (A2), B34.13 (A1), B34.14 (A0), B34.15 (B11), B34.17 (B9), B34.23 (B4), B34.24 (B3), B34.25 (B2), B34.26 (B1), B34.27 (B0), B34.40 (GND), IC15.5 (~{E2}), IC15.8 (GND); no longer B30.21 (B6)
- net RA12: now also B30.33 (Q5); no longer B30.32 (Q4)
- net RA13: now also B30.34 (Q6); no longer B30.33 (Q5)
- net RA14: now also B30.35 (Q7); no longer B30.34 (Q6)
- net VGD0 _{CYCLE 2}: now also B27.27 (B0)
- net VGD1 _{CYCLE 2}: now also B27.26 (B1)
- net VGD2 _{CYCLE 2}: now also B27.25 (B2)
- net VGD3 _{CYCLE 2}: now also B27.24 (B3)
- net VGD4 _{CYCLE 2}: now also B27.23 (B4)
- net VGD5 _{CYCLE 2}: now also B27.22 (B5)
- net VGD6 _{CYCLE 2}: now also B27.21 (B6)
- net VGD7 _{CYCLE 2}: now also B27.19 (B7)
- net VPD0 _{CYCLE 2}: now also B27.18 (B8)
- net VPD1 _{CYCLE 2}: now also B27.17 (B9)
- net VPD2 _{CYCLE 2}: now also B27.16 (B10)
- net VPD3 _{CYCLE 2}: now also B27.15 (B11)
- net VPD4 _{CYCLE 2}: now also B34.22 (B5)
- net VPD5 _{CYCLE 2}: now also B34.21 (B6)
- net VPD6 _{CYCLE 2}: now also B34.19 (B7)
- net VPD7 _{CYCLE 2}: now also B34.18 (B8)
- net ~{Device RAM}: now also IC15.4 (~{E1}); no longer B29.2 (S), B30.2 (S), IC10.2 (1B)
- net ~{RD}: now also B34.3 (A11)
- net ~{RD}·~{WD}: now also IC10.12 (4A), IC10.4 (2A), IC10.9 (3A)
- net ~{WD}: now also B33.2 (T~{DIR}), B34.4 (A10)
- net ~{Device RAM 2}: now reaches IC10.10 (3B)
- net ~{Device RAM 2}: now also IC15.13 (~{Y2})
- net (~{RD}·~{WD})+~{Device RAM 3}: now reaches IC10.11 (4Y)
- net ~{Device RAM 3}: now reaches IC10.13 (4B)
- net ~{Device RAM 3}: now also IC15.12 (~{Y3})
- net ~{Device RAM 1}: now reaches IC10.5 (2B)
- net ~{Device RAM 1}: now also B27.2 (S), B34.2 (S), IC15.14 (~{Y1})
- net (~{RD}·~{WD})+~{Device RAM 1}: now reaches IC10.6 (2Y)
- net (~{RD}·~{WD})+~{Device RAM 2}: now reaches IC10.8 (3Y)
- new net (~{RD}·~{WD})+~{Device RAM 0}: B28.1 (T~{OE}), IC10.3 (1Y)
- new net PA0: B27.28 (Q0), B33.19 (M0)
- new net PA1: B27.29 (Q1), B33.18 (M1)
- new net PA10: B27.38 (Q10), B33.9 (M10)
- new net PA11: B27.39 (Q11), B33.8 (M11)
- new net PA12: B33.7 (M12), B34.33 (Q5)
- new net PA13: B33.6 (M13), B34.34 (Q6)
- new net PA14: B33.5 (M14), B34.35 (Q7)
- new net PA2: B27.30 (Q2), B33.17 (M2)
- new net PA3: B27.31 (Q3), B33.16 (M3)
- new net PA4: B27.32 (Q4), B33.15 (M4)
- new net PA5: B27.33 (Q5), B33.14 (M5)
- new net PA6: B27.34 (Q6), B33.13 (M6)
- new net PA7: B27.35 (Q7), B33.12 (M7)
- new net PA8: B27.36 (Q8), B33.11 (M8)
- new net PA9: B27.37 (Q9), B33.10 (M9)
- new net Palette A Address ~{OE}: B33.3 (M~{OE}), B34.39 (Q11)
- new net Palette A Address ~{WE}: B33.4 (M~{WE}), B34.38 (Q10)
- new net Red0: B33.24 (LQ0)
- new net Red1: B33.25 (LQ1)
- new net Red2: B33.26 (LQ2)
- new net Red3: B33.27 (LQ3)
- new net Red4: B33.28 (LQ4)
- new net Red5: B33.29 (LQ5)
- new net Red6: B33.30 (LQ6)
- new net Red7: B33.31 (LQ7)
- new net ~{Device RAM 0}: B29.2 (S), B30.2 (S), IC10.2 (1B), IC15.15 (~{Y0})
- no-connect marks 96 -> 103
Other:
- moved on the sheet: B28, B29, B30, IC10, IC7, IC8, IC9

Commit message: Added Video memory select boards.
Parts:
- removed B25: Device Decode Stage B, HCP65_Parts:HCP65_Device_Decode_Stage_B, symbol HCP65:Device_Decode_Stage_B
- removed B27, B29, B30, B34: Selector 12bit, HCP65_Parts:HCP65_Selector_12bit, symbol HCP65:Selector_12bit
- removed IC1: 74LVC2G04GW-Q100H, SOP65P210X110-6N, symbol Nexperia:74LVC2G04GW-Q100H
- removed IC10: 74LVC32APW,118, SOP65P640X110-14N, symbol Nexperia:74LVC32APW,118
- removed IC13, IC14: 74LVC574APW,118, SOP65P640X110-20N, symbol Nexperia:74LVC574APW,118
- removed IC15, IC9: 74LVC138APW-Q100J, SOP65P640X110-16N, symbol Nexperia:74LVC138APW-Q100J
- removed IC3, IC7: 74LVC08APW,112, SOP65P640X110-14N, symbol Nexperia:74LVC08APW,112
- removed IC6: 74LVC04APW,118, SOP65P640X110-14N, symbol Nexperia:74LVC04APW,118
- removed IC8: 74LVC163PW,118, SOP65P640X110-16N, symbol Nexperia:74LVC163PW,118
- added B25: Video Device RAM Select, HCP65_Parts:HCP65_Video_Device_RAM_Select, symbol HCP65:Video_Device_RAM_Select
- added B27, B30: Memory 32KB, HCP65_Parts:HCP65_Memory_32KB_With_Latch, symbol HCP65:Memory_32KB
- added B29, B35: Selector 18bit, HCP65_Parts:HCP65_Selector_18bit, symbol HCP65:Selector 18bit
- added B34: Video Main Memory Select, HCP65_Parts:HCP65_Video_Main_Memory_Select, symbol HCP65:Video_Main_Memory_Select
- added C23 (x4): 1μF, SamacSys_Parts:C_0805, symbol HCP65:C_0805
- added C23 (x4): 0.1μF, SamacSys_Parts:C_0805, symbol HCP65:C_0805
- added IC19: TLV702125QDBVRQ1, SOT95P280X145-5N, symbol Texas_Instruments:TLV702125QDBVRQ1
- added IC21, IC22: 74LVC574APW,118, SOP65P640X110-20N, symbol Nexperia:74LVC574APW,118
- added IC23: SN74AHCT74PWR, SOP65P640X110-14N, symbol Texas_Instruments:SN74AHCT74PWR
- added IC5: ADV7125KSTZ50, QFP50P900X900X160-48N, symbol Analog_Devices:ADV7125KSTZ50
- added IC7: 74LVC1G08GV,125, SOT95P275X110-5N, symbol Nexperia:74LVC1G08GV,125
- added R3 (x3): 75Ω, SamacSys_Parts:R_0805, symbol HCP65:R_0805
- added R3: 530Ω, SamacSys_Parts:R_0805, symbol HCP65:R_0805
Connections:
- net (~{RD}·~{WD})+~{Device RAM} is gone; now on net (~{RD}·~{WD})+~{Device RAM 1}: B33.1 (T~{OE})
- net First Pixel _{CYCLE 1H} is gone; now on net Horizontal Sync _{CYCLE 2H}: IC11.12 (Q7), IC12.9 (D7)
- net First Pixel _{CYCLE 1} is gone; now on net Horizontal Sync _{CYCLE 2}: IC12.12 (Q7)
- net First Row _{CYCLE 1H} is gone; now on net Vertical Sync _{CYCLE 2H}: IC11.14 (Q5), IC12.7 (D5)
- net First Row _{CYCLE 1} is gone; now on net Vertical Sync _{CYCLE 2}: IC12.14 (Q5)
- net Last Pixel + 1 _{CYCLE 1H} is gone; now on net Horizontal Blank _{CYCLE 2H}: IC11.13 (Q6), IC12.8 (D6)
- net Last Pixel + 1 _{CYCLE 1} is gone; now on net Horizontal Blank _{CYCLE 2}: IC12.13 (Q6)
- net Last Row + 1 _{CYCLE 1H} is gone; now on net Vertical Blank _{CYCLE 2H}: IC11.15 (Q4), IC12.6 (D4)
- net Last Row + 1 _{CYCLE 1} is gone; now on net Vertical Blank _{CYCLE 2}: IC12.15 (Q4)
- net (~{RD}·~{WD})+~{Device RAM 0}: now also B25.2 ((~{RD}·~{WD})+~{Device_RAM_0})
- net (~{RD}·~{WD})+~{Device RAM 1}: now also B25.3 ((~{RD}·~{WD})+~{Device_RAM_1})
- net (~{RD}·~{WD})+~{Device RAM 2}: now also B25.24 ((~{RD}·~{WD})+~{Device_RAM_2}), B30.1 (T~{OE})
- net (~{RD}·~{WD})+~{Device RAM 3}: now also B25.23 ((~{RD}·~{WD})+~{Device_RAM_3}), B27.1 (T~{OE})
- net 3.3V: now also B29.20 (B16), B35.20 (B16), B35.22 (B14), IC21.20 (3V), IC22.20 (3V), IC5.38 (~{PSAVE}), IC7.5 (3V); no longer B33.22 (LLE)
- net 5V: now also B25.1 (5V), B25.13 (5V), B27.20 (5V), B29.3 (5V), B29.35 (5V), B30.20 (5V), B34.1 (5V), B34.13 (5V), B35.3 (5V), B35.35 (5V), C23.1, C23.1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
- net A0: now also B29.16 (A0), B35.16 (A0)
- net A1: now also B29.15 (A1), B35.15 (A1)
- net A10: now also B29.5 (A10), B35.5 (A10)
- net A11: now also B29.4 (A11), B35.4 (A11)
- net A12: now also B29.2 (A12), B35.2 (A12)
- net A13: now also B29.1 (A13), B35.1 (A13)
- net A14: now also B25.12 (A14), B29.61 (A14), B35.61 (A14)
- net A15: now also B25.11 (A15)
- net A16: now also B25.7 (A16)
- net A2: now also B29.14 (A2), B35.14 (A2)
- net A3: now also B29.13 (A3), B35.13 (A3)
- net A4: now also B29.12 (A4), B35.12 (A4)
- net A5: now also B29.11 (A5), B35.11 (A5)
- net A6: now also B29.9 (A6), B35.9 (A6)
- net A7: now also B29.8 (A7), B35.8 (A7)
- net A8: now also B29.7 (A8), B35.7 (A8)
- net A9: now also B29.6 (A9), B35.6 (A9)
- net D0: now also B27.39 (D7), B30.39 (D7)
- net D1: now also B27.38 (D6), B30.38 (D6)
- net D2: now also B27.37 (D5), B30.37 (D5)
- net D3: now also B27.36 (D4), B30.36 (D4)
- net D4: now also B27.35 (D3), B30.35 (D3)
- net D5: now also B27.34 (D2), B30.34 (D2)
- net D6: now also B27.33 (D1), B30.33 (D1)
- net D7: now also B27.32 (D0), B30.32 (D0)
- net D~{OE}G0: now also B34.20 (D~{OE}G0)
- net D~{OE}G1: now also B34.18 (D~{OE}G1)
- net D~{OE}P0: now also B34.19 (D~{OE}P0)
- net D~{OE}P1: now also B34.17 (D~{OE}P1)
- net First Pixel _{HALF CYCLE}: no longer IC11.9 (D7)
- net First Row _{HALF CYCLE}: no longer IC11.7 (D5)
- net GND: now also B25.16 (GND), B25.21 (GND), B25.4 (GND), B25.9 (GND), B27.21 (GND), B27.23 (L~{OE}), B27.40 (GND), B29.10 (GND), B29.19 (B17), B29.23 (GND), B29.42 (GND), B29.55 (GND)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
- net Horizontal Blank _{CYCLE 1}: now also IC11.8 (D6)
- net Horizontal Blank _{CYCLE 2}: now also IC21.4 (D2)
- net Horizontal Blank _{HALF CYCLE}: now also B34.3 (~{MR})
- net Horizontal Sync _{CYCLE 1}: now also IC11.9 (D7)
- net Horizontal Sync _{CYCLE 2}: now also IC21.5 (D3)
- net LA0: now also B35.33 (B0)
- net LA1: now also B35.34 (B1)
- net Memory Frame: now also B34.8 (Memory_Frame)
- net Pixel CLK: now also B17.6 (Pixel_CLK), B19.40 (CLK), B24.56 (CLK), B26.2 (~{Pixel_CLK}), B33.22 (LLE), B27.22 (LLE), B30.22 (LLE), IC21.11 (CP), IC23.11 (2CP); no longer B22.4 (CLK)
- net RA0: now also B35.41 (Y0)
- net RA1: now also B35.43 (Y1)
- net RA10: now also B35.52 (Y10)
- net RA11: now also B35.53 (Y11)
- net RA12: now also B35.54 (Y12)
- net RA13: now also B35.56 (Y13)
- net RA14: now also B35.57 (Y14)
- net RA2: now also B35.44 (Y2)
- net RA3: now also B35.45 (Y3)
- net RA4: now also B35.46 (Y4)
- net RA5: now also B35.47 (Y5)
- net RA6: now also B35.48 (Y6)
- net RA7: now also B35.49 (Y7)
- net RA8: now also B35.50 (Y8)
- net RA9: now also B35.51 (Y9)
- net Red0: now also IC5.41 (R0)
- net Red1: now also IC5.42 (R1)
- net Red2: now also IC5.43 (R2)
- net Red3: now also IC5.44 (R3)
- net Red4: now also IC5.45 (R4)
- net Red5: now also IC5.46 (R5)
- net Red6: now also IC5.47 (R6)
- net Red7: now also IC5.48 (R7)
- net Row Address ~{OE}: now also B35.60 (Y17)
- net Row Address ~{WE}: now also B35.59 (Y16)
- net Row0: now also B35.36 (B2)
- net Row1: now also B35.37 (B3)
- net Row2: now also B35.38 (B4)
- net Row3: now also B35.32 (B5)
- net Row4: now also B35.31 (B6)
- net Row5: now also B35.30 (B7)
- net Row6: now also B35.29 (B8)
- net Row7: now also B35.28 (B9)
- net Row8: now also B35.27 (B10)
- net Row9: now also B35.26 (B11)
- net VGD0 _{CYCLE 2}: now also B29.33 (B0)
- net VGD1 _{CYCLE 2}: now also B29.34 (B1)
- net VGD2 _{CYCLE 2}: now also B29.36 (B2)
- net VGD3 _{CYCLE 2}: now also B29.37 (B3)
- net VGD4 _{CYCLE 2}: now also B29.38 (B4)
- net VGD5 _{CYCLE 2}: now also B29.32 (B5)
- net VGD6 _{CYCLE 2}: now also B29.31 (B6)
- net VGD7 _{CYCLE 2}: now also B29.30 (B7)
- net VPD0 _{CYCLE 2}: now also B29.29 (B8)
- net VPD1 _{CYCLE 2}: now also B29.28 (B9)
- net VPD2 _{CYCLE 2}: now also B29.27 (B10)
- net VPD3 _{CYCLE 2}: now also B29.26 (B11)
- net VPD4 _{CYCLE 2}: now also B29.25 (B12)
- net VPD5 _{CYCLE 2}: now also B29.24 (B13)
- net VPD6 _{CYCLE 2}: now also B29.22 (B14)
- net VPD7 _{CYCLE 2}: now also B29.21 (B15)
- net Vertical Blank _{CYCLE 1}: now also IC11.6 (D4)
- net Vertical Blank _{CYCLE 2}: now also IC21.2 (D0)
- net Vertical Sync _{CYCLE 1}: now also IC11.7 (D5)
- net Vertical Sync _{CYCLE 2}: now also IC21.3 (D1)
- net ~{Device RAM 0}: now also B25.22 (~{Device_RAM_0}), B35.17 (S)
- net ~{Device RAM}: now also B25.5 (~{Device_RAM}), B29.17 (S)
- net ~{Load Address Bank}: now also B34.24 (~{Load_Address_Low})
- net ~{Load Address High}: now also B34.23 (~{Load_Address_High})
- net ~{Load Address Low}: now also B34.22 (~{Load_Address_Bank})
- net ~{Memory A}: now also B34.6 (~{Memory_A})
- net ~{Memory B}: now also B34.7 (~{Memory_B})
- net ~{Memory Frame}: now also B34.15 (~{Memory_Frame})
- net ~{Pixel CLK}: now also B22.4 (CLK), B34.5 (CLK), IC22.11 (CP), IC23.3 (1CP), IC5.24 (CLK); no longer B17.6 (Pixel_CLK), B19.40 (CLK), B24.56 (CLK), B26.2 (~{Pixel_CLK})
- net ~{RD}: now also B25.8 (~{RD}), B35.64 (A17)
- net ~{WD}: now also B25.10 (~{WD}), B35.63 (A16); no longer B33.2 (T~{DIR})
- net LQ0 renamed Row Address 0
- net LQ1 renamed Row Address 1
- net LQ2 renamed Row Address 2
- net LQ3 renamed Row Address 3
- net LQ4 renamed Row Address 4
- net LQ5 renamed Row Address 5
- net LQ6 renamed Row Address 6
- net LQ7 renamed Row Address 7
- net Last Pixel + 1 renamed Last Pixel+1
- net Last Pixel + 1 _{HALF CYCLE} renamed Last Pixel+1 _{HALF CYCLE}
- net Last Pixel+1 _{HALF CYCLE}: no longer IC11.8 (D6)
- net Last Row + 1 renamed Last Row+1
- net Last Row + 1 _{HALF CYCLE} renamed Last Row+1 _{HALF CYCLE}
- net Last Row+1 _{HALF CYCLE}: no longer IC11.6 (D4)
- net PA0 renamed Palette0
- net Palette0: now also B27.19 (M0), B29.41 (Y0), B30.19 (M0)
- net PA1 renamed Palette1
- net Palette1: now also B27.18 (M1), B29.43 (Y1), B30.18 (M1)
- net PA10 renamed Palette10
- net Palette10: now also B27.9 (M10), B29.52 (Y10), B30.9 (M10)
- net PA11 renamed Palette11
- net Palette11: now also B27.8 (M11), B29.53 (Y11), B30.8 (M11)
- net PA12 renamed Palette12
- net PA13 renamed Palette13
- net PA14 renamed Palette14
- net PA2 renamed Palette2
- net PA3 renamed Palette3
- net PA4 renamed Palette4
- net PA5 renamed Palette5
- net PA6 renamed Palette6
- net PA7 renamed Palette7
- net PA8 renamed Palette8
- net PA9 renamed Palette9
- net Palette A Address ~{OE} renamed ~{RD}+~{Device RAM 1}
- net Palette A Address ~{WE} renamed ~{WD}+~{Device RAM 1}
- new net: C23.1, IC5.35 (Capacitor_{COMP})
- new net: IC5.37 (Resistor_{SET}), R3.1
- new net 1.25V: IC19.5 (OUT), IC5.36 (Voltage_{REF})
- new net Blue _{OUT}: IC5.28 (IOB), R3.1
- new net Blue0: B27.24 (LQ0), IC5.16 (B0)
- new net Blue1: B27.25 (LQ1), IC5.17 (B1)
- new net Blue2: B27.26 (LQ2), IC5.18 (B2)
- new net Blue3: B27.27 (LQ3), IC5.19 (B3)
- new net Blue4: B27.28 (LQ4), IC5.20 (B4)
- new net Blue5: B27.29 (LQ5), IC5.21 (B5)
- new net Blue6: B27.30 (LQ6), IC5.22 (B6)
- new net Blue7: B27.31 (LQ7), IC5.23 (B7)
- new net Green _{OUT}: IC5.32 (IOG), R3.1
- new net Green0: B30.24 (LQ0), IC5.3 (G0)
- new net Green1: B30.25 (LQ1), IC5.4 (G1)
- new net Green2: B30.26 (LQ2), IC5.5 (G2)
- new net Green3: B30.27 (LQ3), IC5.6 (G3)
- new net Green4: B30.28 (LQ4), IC5.7 (G4)
- new net Green5: B30.29 (LQ5), IC5.8 (G5)
- new net Green6: B30.30 (LQ6), IC5.9 (G6)
- new net Green7: B30.31 (LQ7), IC5.10 (G7)
- new net Horizontal Blank _{CYCLE 3H}: IC21.17 (Q2), IC22.4 (D2)
- new net Horizontal Blank _{CYCLE 3}: IC21.8 (D6), IC22.17 (Q2), IC23.2 (1D), IC7.2 (A)
- new net Horizontal Blank _{CYCLE 4H}: IC21.13 (Q6), IC22.8 (D6)
- new net Horizontal Blank _{CYCLE 5}: IC22.13 (Q6)
- new net Horizontal Blank _{OUT}: IC23.5 (1Q)
- new net Horizontal Sync _{CYCLE 3H}: IC21.16 (Q3), IC22.5 (D3)
- new net Horizontal Sync _{CYCLE 3}: IC21.9 (D7), IC22.16 (Q3)
- new net Horizontal Sync _{CYCLE 4H}: IC21.12 (Q7), IC22.9 (D7)
- new net Horizontal Sync _{CYCLE 5}: IC22.12 (Q7)
- new net Red _{OUT}: IC5.34 (IOR), R3.1
- new net Vertical Blank _{CYCLE 3H}: IC21.19 (Q0), IC22.2 (D0)
- new net Vertical Blank _{CYCLE 3}: IC21.6 (D4), IC22.19 (Q0), IC23.12 (2D), IC7.1 (B)
- new net Vertical Blank _{CYCLE 4H}: IC21.15 (Q4), IC22.6 (D4)
- new net Vertical Blank _{CYCLE 5}: IC22.15 (Q4)
- new net Vertical Blank _{OUT}: IC23.9 (2Q)
- new net Vertical Sync _{CYCLE 3H}: IC21.18 (Q1), IC22.3 (D1)
- new net Vertical Sync _{CYCLE 3}: IC21.7 (D5), IC22.18 (Q1)
- new net Vertical Sync _{CYCLE 4H}: IC21.14 (Q5), IC22.7 (D5)
- new net Vertical Sync _{CYCLE 5}: IC22.14 (Q5)
- new net ~{Blank}: IC5.11 (~{BLANK}), IC7.4 (Y)
- new net ~{RD}+~{Device RAM 2}: B25.19 (~{RD}+~{Device_RAM_2}), B30.3 (M~{OE})
- new net ~{RD}+~{Device RAM 3}: B25.18 (~{RD}+~{Device_RAM_3}), B27.3 (M~{OE})
- new net ~{WD}+~{Device RAM 2}: B25.15 (~{WD}+~{Device_RAM_2}), B30.2 (T~{DIR}), B30.4 (M~{WE})
- new net ~{WD}+~{Device RAM 3}: B25.14 (~{WD}+~{Device_RAM_3}), B27.2 (T~{DIR}), B27.4 (M~{WE})
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Other:
- note removed: "Because VA (Video Address) is only latched on ~{Pixel CLK} that means if if VG and VP are also latched on ~{Pixel Clock} then they will still be holding the old values before VA changes."
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