File: Kicad/Computer/Video/Video Board/Video Board.kicad_sch (KiCad schematic)
At the start: 71 parts, among them IC1 LD1117S50C, IC11 74LVC574APW,118, IC12 74LVC574APW,118, IC19 TLV702125QDBVRQ1, IC2 SST39VF010-70-4I-NHE, IC21 74LVC574APW,118, IC22 74LVC574APW,118, IC23 SN74AHCT74PWR, IC27 74LVC1GX04GW,125, IC5 ADV7125KSTZ50, IC7 74LVC1G08GV,125, J5 395-098-520-350

Commit message: Added a Video DAC and a Video Signal Dragger.
Parts:
- removed C23 (x4): 1μF, SamacSys_Parts:C_0805, symbol HCP65:C_0805
- removed C23 (x4): 0.1μF, SamacSys_Parts:C_0805, symbol HCP65:C_0805
- removed IC19: TLV702125QDBVRQ1, SOT95P280X145-5N, symbol Texas_Instruments:TLV702125QDBVRQ1
- removed IC23: SN74AHCT74PWR, SOP65P640X110-14N, symbol Texas_Instruments:SN74AHCT74PWR
- removed IC5: ADV7125KSTZ50, QFP50P900X900X160-48N, symbol Analog_Devices:ADV7125KSTZ50
- removed IC7: 74LVC1G08GV,125, SOT95P275X110-5N, symbol Nexperia:74LVC1G08GV,125
- removed R3 (x3): 75Ω, SamacSys_Parts:R_0805, symbol HCP65:R_0805
- removed R3: 530Ω, SamacSys_Parts:R_0805, symbol HCP65:R_0805
- added B36: Video DAC, HCP65_Parts:HCP65_Video_DAC, symbol HCP65:Video_DAC
- added B38: D-type Flip Flop 24bit, HCP65_Parts:HCP65_D_Flip_Flop_24bit, symbol HCP65:D_Flip_Flop_24bit
Connections:
- net 5V: now also B36.23 (5V), B36.3 (5V), B38.3 (5V), B38.31 (5V)
- net Blue0: now also B38.28 (IN0)
- net Blue1: now also B38.27 (IN1)
- net Blue2: now also B38.26 (IN2)
- net Blue3: now also B38.25 (IN3)
- net Blue4: now also B38.24 (IN4)
- net Blue5: now also B38.23 (IN5)
- net Blue6: now also B38.22 (IN6)
- net Blue7: now also B38.21 (IN7)
- net GND: now also B36.14 (GND), B36.27 (GND), B36.34 (GND), B36.7 (GND), B38.1 (~{OE}), B38.10 (GND), B38.20 (GND), B38.37 (GND), B38.47 (GND)
- net Green0: now also B38.19 (IN8)
- net Green1: now also B38.18 (IN9)
- net Green2: now also B38.17 (IN10)
- net Green3: now also B38.16 (IN11)
- net Green4: now also B38.15 (IN12)
- net Green5: now also B38.14 (IN13)
- net Green6: now also B38.13 (IN14)
- net Green7: now also B38.12 (IN15)
- net Horizontal Blank _{CYCLE 4H}: now also B36.2 (Horizontal_Blank)
- net Horizontal Sync _{CYCLE 4H}: now also B36.4 (Horizontal_Sync)
- net Pixel CLK: now also B36.6 (~{CLK}), B38.56 (CLK)
- net Red0: now also B38.11 (IN16)
- net Red1: now also B38.9 (IN17)
- net Red2: now also B38.8 (IN18)
- net Red3: now also B38.7 (IN19)
- net Red4: now also B38.6 (IN20)
- net Red5: now also B38.5 (IN21)
- net Red6: now also B38.4 (IN22)
- net Red7: now also B38.2 (IN23)
- net Vertical Blank _{CYCLE 4H}: now also B36.10 (Vertical_Blank)
- net Vertical Sync _{CYCLE 4H}: now also B36.11 (Vertical_Sync)
- net ~{Pixel CLK}: now also B36.8 (CLK)
- net Horizontal Blank _{CYCLE 5} renamed Horizontal Blank _{CYCLE 4}
- net Horizontal Sync _{CYCLE 5} renamed Horizontal Sync _{CYCLE 4}
- net Vertical Blank _{CYCLE 5} renamed Vertical Blank _{CYCLE 4}
- net Vertical Sync _{CYCLE 5} renamed Vertical Sync _{CYCLE 4}
- new net Blue0 _{HALF CYCLE}: B36.20 (Blue0), B38.29 (OUT0)
- new net Blue1 _{HALF CYCLE}: B36.19 (Blue1), B38.30 (OUT1)
- new net Blue2 _{HALF CYCLE}: B36.18 (Blue2), B38.32 (OUT2)
- new net Blue3 _{HALF CYCLE}: B36.17 (Blue3), B38.33 (OUT3)
- new net Blue4 _{HALF CYCLE}: B36.16 (Blue4), B38.34 (OUT4)
- new net Blue5 _{HALF CYCLE}: B36.15 (Blue5), B38.35 (OUT5)
- new net Blue6 _{HALF CYCLE}: B36.13 (Blue6), B38.36 (OUT6)
- new net Blue7 _{HALF CYCLE}: B36.12 (Blue7), B38.38 (OUT7)
- new net Green0 _{HALF CYCLE}: B36.32 (Green0), B38.39 (OUT8)
- new net Green1 _{HALF CYCLE}: B36.33 (Green1), B38.40 (OUT9)
- new net Green2 _{HALF CYCLE}: B36.35 (Green2), B38.41 (OUT10)
- new net Green3 _{HALF CYCLE}: B36.36 (Green3), B38.42 (OUT11)
- new net Green4 _{HALF CYCLE}: B36.37 (Green4), B38.43 (OUT12)
- new net Green5 _{HALF CYCLE}: B36.38 (Green5), B38.44 (OUT13)
- new net Green6 _{HALF CYCLE}: B36.39 (Green6), B38.45 (OUT14)
- new net Green7 _{HALF CYCLE}: B36.40 (Green7), B38.46 (OUT15)
- new net Red0 _{HALF CYCLE}: B36.21 (Red0), B38.48 (OUT16)
- new net Red1 _{HALF CYCLE}: B36.22 (Red1), B38.49 (OUT17)
- new net Red2 _{HALF CYCLE}: B36.24 (Red2), B38.50 (OUT18)
- new net Red3 _{HALF CYCLE}: B36.25 (Red3), B38.51 (OUT19)
- new net Red4 _{HALF CYCLE}: B36.26 (Red4), B38.52 (OUT20)
- new net Red5 _{HALF CYCLE}: B36.28 (Red5), B38.53 (OUT21)
- new net Red6 _{HALF CYCLE}: B36.29 (Red6), B38.54 (OUT22)
- new net Red7 _{HALF CYCLE}: B36.30 (Red7), B38.55 (OUT23)
- no-connect marks 73 -> 71
Other:
- note added: "VP.. and VG.. are latched on CLK rising and are valid on ~{CLK}. Therefor Palette.. is valid on ~{CLK}"
