File: Kicad/Computer/MPU/HCP65 Kernal Mode/HCP65 Kernal Mode.kicad_sch (KiCad schematic)
At the start: 26 parts, among them IC1 74F269D, IC2 74LVC02APW,118, IC2 AP7365-33WG-7, IC3 SN74F521NSR, IC4 74LVC16244ADGG,112, IC5 74LVC02APW,118, IC5 74LVC04APW,118, IC6 74LVC04APW,118, IC7 74LVC16373ADL,118, IC8 74LVC541APW,118, J1 Pin_Header_01x32, J2 Conn_02x32_Counter_Clockwise, J3 Pin_Header_01x32

Commit message: Split Kernal Mode into the kernal counter and instruction code.
Parts:
- removed C27: 1μF, SamacSys_Parts:C_0805, symbol HCP65:C_0805
- removed IC1: 74F269D, SamacSys_Parts:SOIC127P1032X265-24N, symbol Nexperia:74F269D
- removed IC2: 74LVC02APW,118, SOP65P640X110-14N, symbol Nexperia:74LVC02APW,118_Multi
- removed unit 4 of IC2
- removed unit 2 of IC2
- removed unit 3 of IC2
- removed IC3: SN74F521NSR, SOIC127P780X200-20N, symbol Texas_Instruments:SN74F521NSR
- removed IC4: 74LVC16244ADGG,112, 74LVC16244ADGG112, symbol Nexperia:74LVC16244ADGG,112
- removed unit 6 of IC5
- removed unit 4 of IC5
- removed unit 2 of IC5
- removed unit 5 of IC5
- removed unit 3 of IC5
- added C27 (x3): 1μF, SamacSys_Parts:C_0805, symbol HCP65:C_0805
- added IC1: 74LVC1G02GV,125, SOT95P275X110-5N, symbol Nexperia:74LVC1G02GV,125
- added IC12: 74LVC138APW-Q100J, SOP65P640X110-16N, symbol Nexperia:74LVC138APW-Q100J
- added IC2: 74LVC11PW,112, SOP65P640X110-14N, symbol Nexperia:74LVC11PW,112
- added IC3: 74LVC32APW,118, SOP65P640X110-14N, symbol Nexperia:74LVC32APW,118_Multi
- added IC4: 74LVC16244ADGG,112, 74LVC16244ADGG112, symbol Nexperia:74LVC16244ADGG,112_Multi
- added IC5, IC9: 74HCT193PW,118, SOP65P640X110-16N, symbol Nexperia:74HCT193PW,118
- added TP1, TP2: TestPoint, Connector_PinHeader_2.54mm:PinHeader_1x01_P2.54mm_Vertical, symbol Connector:TestPoint
Connections:
- net C7 is gone; now on net C2: J2.14 (Pin_14)
- net 3.3V: now also C27.2, C27.2, IC1.5 (3V), IC12.16 (3V), IC2.14 (3V), IC3.14 (3V), IC3.14 (3V), IC3.14 (3V), IC3.14 (3V), IC4.18 (3V), IC4.31 (3V), IC4.42 (3V), IC4.7 (3V)
- net 5V: now also C27.2, IC5.16 (5V), IC9.16 (5V)
- net A_{OUT}16: now also J2.50 (Pin_50); no longer J2.53 (Pin_53)
- net A_{OUT}17: now also J2.49 (Pin_49); no longer J2.52 (Pin_52)
- net A_{OUT}18: now also J2.48 (Pin_48); no longer J2.51 (Pin_51)
- net A_{OUT}19: now also J2.47 (Pin_47); no longer J2.50 (Pin_50)
- net A_{OUT}20: now also J2.46 (Pin_46); no longer J2.49 (Pin_49)
- net A_{OUT}21: now also J2.45 (Pin_45); no longer J2.48 (Pin_48)
- net A_{OUT}22: now also J2.44 (Pin_44); no longer J2.47 (Pin_47)
- net A_{OUT}23: now also J2.43 (Pin_43); no longer J2.46 (Pin_46)
- net C0: now also J2.12 (Pin_12), IC2.1 (1A), IC4.36 (3A0), IC9.7 (Q3); no longer J2.6 (Pin_6)
- net C1: now also J2.13 (Pin_13), IC2.2 (1B), IC4.35 (3A1), IC9.6 (Q2); no longer J2.7 (Pin_7)
- net C2: now also IC2.13 (1C), IC4.33 (3A2), IC9.2 (Q1); no longer J2.8 (Pin_8)
- net C3: now also J2.52 (Pin_52), IC2.3 (2A), IC4.32 (3A3), IC9.3 (Q0); no longer J2.9 (Pin_9)
- net C4: now also J2.51 (Pin_51), IC2.4 (2B), IC4.30 (4A0), IC5.3 (Q0); no longer J2.11 (Pin_11)
- net C5: now also IC2.5 (2C), IC4.29 (4A1), IC5.2 (Q1), TP2.1; no longer J2.12 (Pin_12)
- net C6: now also IC2.9 (3A), IC4.27 (4A2), IC5.6 (Q2), TP1.1; no longer J2.13 (Pin_13)
- net D0: now also IC4.13 (3Y0), IC4.2 (1Y0), IC9.15 (D0)
- net D1: now also IC4.14 (3Y1), IC4.3 (1Y1), IC9.1 (D1)
- net D2: now also IC4.16 (3Y2), IC4.5 (1Y2), IC9.10 (D2)
- net D3: now also IC4.17 (3Y3), IC4.6 (1Y3), IC9.9 (D3)
- net D4: now also IC4.19 (4Y0), IC4.8 (2Y0), IC5.15 (D0)
- net D5: now also IC4.20 (4Y1), IC4.9 (2Y1), IC5.1 (D1)
- net D6: now also IC4.11 (2Y2), IC4.22 (4Y2), IC5.10 (D2)
- net D7: now also IC4.12 (2Y3), IC4.23 (4Y3), IC5.9 (D3)
- net Enter Interrupt: now also IC6.12 (6Y), J2.56 (Pin_56), IC9.5 (CPU); no longer J2.62 (Pin_62)
- net GND: now also C27.1, C27.1, C27.1, IC1.3 (GND), IC12.8 (GND), IC2.7 (GND), IC3.10 (3B), IC3.7 (GND), IC3.7 (GND), IC3.7 (GND), IC3.7 (GND), IC3.9 (3A), IC4.10 (GND), IC4.15 (GND), IC4.21 (GND), IC4.26 (4A3), IC4.28 (GND), IC4.34 (GND), IC4.39 (GND), IC4.4 (GND), IC4.45 (GND), IC5.8 (GND), IC9.8 (GND); no longer IC6.1 (1A), IC6.13 (6A)
- net Kernal Mode: now also IC6.5 (3A), J2.53 (Pin_53), IC1.4 (Y); no longer IC6.3 (2A), J2.56 (Pin_56)
- net Kernal Mode_{ PART}: now also IC6.3 (2A), IC2.8 (3Y); no longer IC6.5 (3A), J2.61 (Pin_61)
- net Native Latch: now also IC1.1 (B)
- net RTI: now also IC6.2 (1Y), J2.11 (Pin_11), IC9.4 (CPD); no longer J2.63 (Pin_63)
- net ~{Interrupt Depth}: now also J2.9 (Pin_9), IC3.12 (4A); no longer J2.59 (Pin_59)
- net ~{Kernal Mode}: now also IC6.6 (3Y), J2.54 (Pin_54); no longer IC6.4 (2Y), J2.57 (Pin_57)
- net ~{Kernal Mode}_{ PART}: now also IC6.4 (2Y), IC1.2 (A); no longer IC6.6 (3Y)
- net ~{RD}: now also J2.6 (Pin_6); no longer J2.58 (Pin_58)
- net ~{RTI}: now also IC6.1 (1A), IC12.15 (~{Y0})
- net ~{Read Interrupt Depth}: now also IC4.24 (4~{OE}), IC4.25 (3~{OE})
- net ~{VP}: now also IC6.13 (6A)
- net ~{WD}: now also J2.7 (Pin_7), IC3.13 (4B); no longer J2.54 (Pin_54)
- net Interrupt CLK renamed ~{Reset}
- net ~{Reset}: now also IC5.14 (MR), IC9.14 (MR)
- net Opcode Valid renamed OP7
- net OP7: now also IC3.1 (1A)
- net Read User Program renamed Read Process ID
- net UP0 renamed PID0
- net PID0: now also IC4.47 (1A0)
- net UP1 renamed PID1
- net PID1: now also IC4.46 (1A1)
- net UP2 renamed PID2
- net PID2: now also IC4.44 (1A2)
- net UP3 renamed PID3
- net PID3: now also IC4.43 (1A3)
- net UP4 renamed PID4
- net PID4: now also IC4.41 (2A0)
- net UP5 renamed PID5
- net PID5: now also IC4.40 (2A1)
- net UP6 renamed PID6
- net PID6: now also IC4.38 (2A2)
- net UP7 renamed PID7
- net PID7: now also IC4.37 (2A3)
- net Write Interrupt Depth: no longer names the net of IC5.11 (4Y)
- net Write User Program renamed Write Process ID
- net ~{Read User Program} renamed ~{Read Process ID}
- net ~{Read Process ID}: now also IC4.1 (1~{OE}), IC4.48 (2~{OE})
- net ~{User Program} renamed ~{Process ID}
- net ~{Process ID}: now also J2.8 (Pin_8); no longer J2.60 (Pin_60)
- new net: IC12.4 (~{E1}), IC3.3 (1Y)
- new net: IC12.5 (~{E2}), IC3.6 (2Y)
- new net C0⋅C1⋅C2: IC2.10 (3B), IC2.12 (1Y)
- new net C3⋅C4⋅C5: IC2.11 (3C), IC2.6 (2Y)
- new net OP0: IC12.1 (A0), J2.57 (Pin_57)
- new net OP1: IC12.2 (A1), J2.58 (Pin_58)
- new net OP2: IC12.3 (A2), J2.59 (Pin_59)
- new net OP3: IC3.5 (2B), J2.60 (Pin_60)
- new net OP4: IC3.4 (2A), J2.61 (Pin_61)
- new net OP5: IC3.2 (1B), J2.62 (Pin_62)
- new net OP6: IC12.6 (E3), J2.63 (Pin_63)
- new net ~{TCD}: IC5.4 (CPD), IC9.13 (~{TCD})
- new net ~{TCU}: IC5.5 (CPU), IC9.12 (~{TCU})
- new net ~{Write Interrupt Depth}: IC3.11 (4Y), IC5.11 (~{PL}), IC9.11 (~{PL})
- no-connect marks 7 -> 14
Other:
- moved on the sheet: C27, IC6A, IC6B, IC6C, IC6E, IC6F

Commit message: Re-routed Kernal Mode board.
Parts:
- removed IC7: 74LVC16373ADL,118, SOP64P1025X280-48N, symbol Nexperia:74LVC16373ADL,118
- added IC7: 74LVC16373ADL,118, SOP64P1025X280-48N, symbol Nexperia:74LVC16373ADL,118_Multi
Connections:
- net 3.3V: now also IC7.18 (3V), IC7.31 (3V), IC7.42 (3V), IC7.7 (3V)
- net A_{OUT}16: now also IC7.2 (1Q0)
- net A_{OUT}17: now also IC7.3 (1Q1)
- net A_{OUT}18: now also IC7.5 (1Q2)
- net A_{OUT}19: now also IC7.6 (1Q3)
- net A_{OUT}20: now also IC7.8 (1Q4)
- net A_{OUT}21: now also IC7.9 (1Q5)
- net A_{OUT}22: now also IC7.11 (1Q6)
- net A_{OUT}23: now also IC7.12 (1Q7)
- net D0: now also IC7.36 (2D0), IC7.47 (1D0)
- net D1: now also IC7.35 (2D1), IC7.46 (1D1)
- net D2: now also IC7.33 (2D2), IC7.44 (1D2)
- net D3: now also IC7.32 (2D3), IC7.43 (1D3)
- net D4: now also IC7.30 (2D4), IC7.41 (1D4)
- net D5: now also IC7.29 (2D5), IC7.40 (1D5)
- net D6: now also IC7.27 (2D6), IC7.38 (1D6)
- net D7: now also IC7.26 (2D7), IC7.37 (1D7)
- net GND: now also IC7.10 (GND), IC7.15 (GND), IC7.21 (GND), IC7.24 (2~{OE}), IC7.28 (GND), IC7.34 (GND), IC7.39 (GND), IC7.4 (GND), IC7.45 (GND)
- net Kernal Mode: now also IC7.1 (1~{OE})
- net Latch Bank Remap: now also IC7.48 (1LE)
- net PID0: now also IC7.13 (2Q0)
- net PID1: now also IC7.14 (2Q1)
- net PID2: now also IC7.16 (2Q2)
- net PID3: now also IC7.17 (2Q3)
- net PID4: now also IC7.19 (2Q4)
- net PID5: now also IC7.20 (2Q5)
- net PID6: now also IC7.22 (2Q6)
- net PID7: now also IC7.23 (2Q7)
- net Write Process ID: now also IC7.25 (2LE)
- net C0⋅C1⋅C2 renamed C0·C1·C2
- net C3⋅C4⋅C5 renamed C3·C4·C5
Other:
- moved on the sheet: IC3C, IC4A, IC4B, IC6D, IC6E

Commit message: Use thinner boards for Video components.
Changed lines of the file:
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@@
     (effects (font (size 1.27 1.27)) (justify right bottom))
   )
-  (label "D3" (at 396.24 370.84 0) (fields_autoplaced)
+  (label "D3" (at 396.24 373.38 0) (fields_autoplaced)
     (effects (font (size 1.27 1.27)) (justify left bottom))
   )
@@
     (effects (font (size 1.27 1.27) italic) (justify left bottom))
   )
-  (label "D0" (at 396.24 342.9 0) (fields_autoplaced)
+  (label "D0" (at 396.24 345.44 0) (fields_autoplaced)
     (effects (font (size 1.27 1.27)) (justify left bottom))
   )
@@
     (effects (font (size 1.27 1.27)) (justify right bottom))
   )
-  (label "D1" (at 396.24 340.36 0) (fields_autoplaced)
+  (label "D1" (at 396.24 342.9 0) (fields_autoplaced)
     (effects (font (size 1.27 1.27)) (justify left bottom))
   )
@@
     (effects (font (size 1.27 1.27)) (justify left bottom))
   )
-  (label "D1" (at 396.24 375.92 0) (fields_autoplaced)
+  (label "D1" (at 396.24 378.46 0) (fields_autoplaced)
     (effects (font (size 1.27 1.27)) (justify left bottom))
   )
@@
     (effects (font (size 1.27 1.27)) (justify right bottom))
   )
-  (label "D3" (at 396.24 335.28 0) (fields_autoplaced)
+  (label "D3" (at 396.24 337.82 0) (fields_autoplaced)
     (effects (font (size 1.27 1.27)) (justify left bottom))
   )
@@
     (effects (font (size 1.27 1.27)) (justify right bottom))
   )
-  (label "D2" (at 396.24 337.82 0) (fields_autoplaced)
+  (label "D2" (at 396.24 340.36 0) (fields_autoplaced)
     (effects (font (size 1.27 1.27)) (justify left bottom))
   )
@@
     (effects (font (size 1.27 1.27)) (justify right bottom))
   )
-  (label "D2" (at 396.24 373.38 0) (fields_autoplaced)
+  (label "D2" (at 396.24 375.92 0) (fields_autoplaced)
     (effects (font (size 1.27 1.27)) (justify left bottom))
   )
@@
     (effects (font (size 1.27 1.27)) (justify right bottom))
   )
-  (label "D0" (at 396.24 378.46 0) (fields_autoplaced)
+  (label "D0" (at 396.24 381 0) (fields_autoplaced)
     (effects (font (size 1.27 1.27)) (justify left bottom))
   )
@@
     )
   )
-  (symbol (lib_id "Nexperia:74LVC16244ADGG,112_Multi") (at 370.84 332.74 0) (unit 1)
+  (symbol (lib_name "74LVC16244ADGG,112_Multi_2") (lib_id "Nexperia:74LVC16244ADGG,112_Multi") (at 370.84 332.74 0) (unit 1)
     (in_bom yes) (on_board yes) (dnp no)
     (property "Reference" "IC4" (at 383.54 327.025 0)
@@
     )
   )
-  (symbol (lib_id "Nexperia:74LVC16244ADGG,112_Multi") (at 370.84 368.3 0) (unit 2)
+  (symbol (lib_name "74LVC16244ADGG,112_Multi_1") (lib_id "Nexperia:74LVC16244ADGG,112_Multi") (at 370.84 368.3 0) (unit 2)
     (in_bom yes) (on_board yes) (dnp no)
     (property "Reference" "IC4" (at 383.54 362.585 0)

Commit message: Regenerating some gerbers again with paste layers.  Fixed Address Decode Wide.
Other:
- title: (none) -> Kernal Mode
- moved on the sheet: C27, IC1, IC12, IC2, IC3A, IC3B, IC3C, IC3D, IC4A, IC4B, IC4C, IC5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

Commit message: Added Video Palette (Memory B) writing.
Parts:
- IC1: footprint SOT95P275X110-5N -> SamacSys_Parts:SOT95P275X110-5N; Garbage (none) -> 74LVC1G02 - Single 2-input NOR gate@en-us
- IC12: footprint SOP65P640X110-16N -> SamacSys_Parts:SOP65P640X110-16N; Garbage (none) -> 74LVC138A-Q100 - 3-to-8 line decoder/demultiplexer; inverti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
- IC2: footprint SOT95P285X130-5N -> SamacSys_Parts:SOT95P285X130-5N; Garbage (none) -> DiodesZetex AP7365-33WG-7, LDO Voltage Regulator, 600mA, 3.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
- IC2: footprint SOP65P640X110-14N -> SamacSys_Parts:SOP65P640X110-14N; Garbage (none) -> 74LVC11 - Triple 3-input AND gate@en-us
- IC3: footprint SOP65P640X110-14N -> SamacSys_Parts:SOP65P640X110-14N; Garbage (none) -> 74LVC32A - Quad 2-input OR gate@en-us
- IC4: footprint 74LVC16244ADGG112 -> SamacSys_Parts:74LVC16244ADGG112; Garbage (none) -> 74LVC16244A; 74LVCH16244A - 16-bit buffer/line driver; 5 V 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
- IC5: footprint SOP65P640X110-14N -> SamacSys_Parts:SOP65P640X110-14N; Garbage (none) -> Nexperia 74LVC02APW,118, Quad 2-Input NOR Logic Gate, 14-Pi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
- IC5, IC9: footprint SOP65P640X110-16N -> SamacSys_Parts:SOP65P640X110-16N; Garbage (none) -> 74HC(T)193 - Presettable synchronous 4-bit binary up, down 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
- IC6: footprint SOP65P640X110-14N -> SamacSys_Parts:SOP65P640X110-14N; Garbage (none) -> 74LVC04A - Hex inverter@en-us
- IC7: footprint SOP64P1025X280-48N -> SamacSys_Parts:SOP64P1025X280-48N; Garbage (none) -> 74LVC16373A; 74LVCH16373A - 16-bit D-type transparent latch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
- IC8: footprint SOP65P640X110-20N -> SamacSys_Parts:SOP65P640X110-20N; Garbage (none) -> 74LVC541A - Octal buffer/line driver with 5 V tolerant inpu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

Commit message: Converted more PCBs to Kicad 8.
Parts:
- C27: Garbage (none) -> Unpolarized capacitor, small symbol
- IC4: Garbage 74LVC16244A; 74LVCH16244A - 16-bit buffer/line driver; 5 V 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 -> (none)
- IC7: Garbage 74LVC16373A; 74LVCH16373A - 16-bit D-type transparent latch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 -> (none)
Other:
- moved on the sheet: TP1, TP2
