File: Kicad/Temp/Latch Slow/Latch Slow.kicad_sch (KiCad schematic)
At the start: 15 parts, among them IC1 SN74AHCT08PWRG4, J1 Conn_01x01_Pin, J2 Conn_01x01_Pin, J3 Conn_01x01_Pin, J4 Conn_01x01_Pin, J5 Conn_01x01_Pin

Commit message: Added a (potentially) 50MHz board.
Parts:
- IC1: footprint SOP65P640X120-14N -> SamacSys_Parts:SOP65P640X120-14N; Garbage (none) -> Logic Gates Quadruple 2-Input Positive-AND Gates
- J1, J2, J3, J4, J5: footprint SamacSys_Parts:Plated_Hole_D1.0mm -> (none)
