File: Kicad/Computer/Component Boards/Counter 16bit with IO/Counter 16bit with IO.kicad_pcb (KiCad board)
At the start: 2 copper layers, 26.7 x 59.7 mm, 24 parts, among them IC1 74LVC573APW,118, IC10 74LVC161PW,112, IC11 74LVC574APW,118, IC12 74LVC574APW,118, IC2 74LVC573APW,118, IC3 74LVC1G08GV,125, IC4 74LVC2G04GW-Q100H, IC5 AP7365-33WG-7, IC7 74LVC161PW,112, IC8 74LVC161PW,112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

Commit message: Started adding Graphics Board.
Connections:
- net CE renamed Count Enable
- net CP renamed CLK
- net ~{MR} renamed ~{Reset}
- net ~{PE} renamed ~{Load Count Start}
Changed lines of the file:
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@@
 	(net 34 "Read Address High")
 	(net 35 "C1")
-	(net 36 "~{PE}")
+	(net 36 "~{Load Count Start}")
 	(net 37 "unconnected-(IC5-ADJ-Pad4)")
-	(net 38 "CE")
+	(net 38 "Count Enable")
 	(net 39 "C0")
 	(net 40 "C2")
-	(net 41 "~{MR}")
+	(net 41 "~{Reset}")
 	(net 42 "C3")
-	(net 43 "CP")
+	(net 43 "CLK")
 	(net 44 "C4")
 	(net 45 "C5")
@@
 			(size 0.45 1.45)
 			(layers "F.Cu" "F.Paste" "F.Mask")
-			(net 41 "~{MR}")
+			(net 41 "~{Reset}")
 			(pinfunction "~{MR}")
 			(pintype "input")
@@
 			(size 0.45 1.45)
 			(layers "F.Cu" "F.Paste" "F.Mask")
-			(net 43 "CP")
+			(net 43 "CLK")
 			(pinfunction "CP")
 			(pintype "input")
@@
 			(size 0.45 1.45)
 			(layers "F.Cu" "F.Paste" "F.Mask")
-			(net 38 "CE")
+			(net 38 "Count Enable")
 			(pinfunction "CEP")
 			(pintype "input")
@@
 			(size 0.45 1.45)
 			(layers "F.Cu" "F.Paste" "F.Mask")
-			(net 36 "~{PE}")
+			(net 36 "~{Load Count Start}")
 			(pinfunction "~{PE}")
 			(pintype "input")
@@
 			(size 0.45 1.45)
 			(layers "F.Cu" "F.Paste" "F.Mask")
-			(net 41 "~{MR}")
+			(net 41 "~{Reset}")
 			(pinfunction "~{MR}")
 			(pintype "input")
@@
 			(size 0.45 1.45)
 			(layers "F.Cu" "F.Paste" "F.Mask")
-			(net 43 "CP")
+			(net 43 "CLK")
 			(pinfunction "CP")
 			(pintype "input")
@@
 			(size 0.45 1.45)
 			(layers "F.Cu" "F.Paste" "F.Mask")
-			(net 36 "~{PE}")
+			(net 36 "~{Load Count Start}")
 			(pinfunction "~{PE}")
 			(pintype "input")
@@
 			(size 0.45 1.45)
 			(layers "F.Cu" "F.Paste" "F.Mask")
-			(net 41 "~{MR}")
+			(net 41 "~{Reset}")
 			(pinfunction "~{MR}")
 			(pintype "input")
@@
 			(size 0.45 1.45)
 			(layers "F.Cu" "F.Paste" "F.Mask")
-			(net 43 "CP")
+			(net 43 "CLK")
 			(pinfunction "CP")
 			(pintype "input")
@@
 			(size 0.45 1.45)
 			(layers "F.Cu" "F.Paste" "F.Mask")
-			(net 36 "~{PE}")
+			(net 36 "~{Load Count Start}")
 			(pinfunction "~{PE}")
 			(pintype "input")
@@
 			(size 0.45 1.45)
 			(layers "F.Cu" "F.Paste" "F.Mask")
-			(net 41 "~{MR}")
+			(net 41 "~{Reset}")
 			(pinfunction "~{MR}")
 			(pintype "input")
@@
 			(size 0.45 1.45)
 			(layers "F.Cu" "F.Paste" "F.Mask")
-			(net 43 "CP")
+			(net 43 "CLK")
 			(pinfunction "CP")
 			(pintype "input")
@@
 			(size 0.45 1.45)
 			(layers "F.Cu" "F.Paste" "F.Mask")
-			(net 36 "~{PE}")
+			(net 36 "~{Load Count Start}")
 			(pinfunction "~{PE}")
 			(pintype "input")
@@
 			(layers "*.Cu" "*.Mask")
 			(remove_unused_layers no)
-			(net 43 "CP")
+			(net 43 "CLK")
 			(pinfunction "Pin_4")
 			(pintype "passive")
@@
 			(layers "*.Cu" "*.Mask")
 			(remove_unused_layers no)
-			(net 36 "~{PE}")
+			(net 36 "~{Load Count Start}")
 			(pinfunction "Pin_5")
 			(pintype "passive")
@@
 			(layers "*.Cu" "*.Mask")
 			(remove_unused_layers no)
-			(net 41 "~{MR}")
+			(net 41 "~{Reset}")
 			(pinfunction "Pin_6")
 			(pintype "passive")
@@
 			(layers "*.Cu" "*.Mask")
 			(remove_unused_layers no)
-			(net 38 "CE")
+			(net 38 "Count Enable")
 			(pinfunction "Pin_17")
 			(pintype "passive")
